Commit message: Mouvement du cou principalement et changement dans le urdf

File: sara_description/urdf/sara.urdf (robot description, URDF)
Before this commit: robot sara, 15 links, 14 joints
Links:
- removed link base_laser_link
- removed link sara_base
- added link laser_link, mass 0.5; collision cylinder length=0.1 radius=0.03; visual cylinder length=0.1 radius=0.03
- added link neckHead_dynamixel_link; visual cylinder length=0.015 radius=0.02
- added link real_base_link, mass 10; collision box size=0.55 0.64311 0.57; collision box size=0.7637 0.64311 0.14
- link base_link: mass 10 -> None; geometry visual box size=0.7637 0.64311 0.14
- link camera_link: geometry visual mesh filename=package://sara_description/meshes/xtion.STL scale=0.001 0.001 0.001
- link clavicule_link: geometry collision mesh filename=package://sara_description/meshes/epaule.STL scale=0.001 0.001 0.001; visual mesh filename=package://sara_description/meshes/epaule.STL scale=0.001 0.001 0.001
- link fixLowerArm_link: geometry collision mesh filename=package://sara_description/meshes/coude.STL scale=0.001 0.001 0.001; visual mesh filename=package://sara_description/meshes/coude.STL scale=0.001 0.001 0.001
- link fixUpperArm_link: geometry collision mesh filename=package://sara_description/meshes/epaule.STL scale=0.001 0.001 0.001; visual mesh filename=package://sara_description/meshes/epaule.STL scale=0.001 0.001 0.001
- link head_link: geometry collision sphere radius=0.1; visual mesh filename=package://sara_description/meshes/tete.STL scale=0.001 0.001 0.001
- link neck_link: geometry visual mesh filename=package://sara_description/meshes/cou.STL scale=0.001 0.001 0.001
- link rotLowerArm_link: geometry collision mesh filename=package://sara_description/meshes/pince-avant-bras.STL scale=0.001 0.001 0.001; visual mesh filename=package://sara_description/meshes/pince-avant-bras.STL scale=0.001 0.001 0.001
- link rotUpperArm_link: geometry collision mesh filename=package://sara_description/meshes/bras_haut.STL scale=0.001 0.001 0.001; visual mesh filename=package://sara_description/meshes/bras_haut.STL scale=0.001 0.001 0.001
- link torso_link: geometry collision mesh filename=package://sara_description/meshes/torse.STL scale=0.001 0.001 0.001; visual mesh filename=package://sara_description/meshes/torse.STL scale=0.001 0.001 0.001
Joints:
- added joint neckHead_dynamixel_joint: type revolute, parent head_link, child neckHead_dynamixel_link, origin xyz=0 -0.054 0 rpy=0 0 0, axis 0 0 1, limit lower=-1.5 upper=1.5 effort=1000.0 velocity=0.5
- joint base_revolute_joint: child base_link -> real_base_link
- joint base_spine_joint: parent base_link -> real_base_link
- joint base_x_trans_joint: parent sara_base -> base_link
- joint camera_joint: origin xyz=0.075 -0.09 0 rpy=1.57 0 0 -> xyz=0.0776104 -0.13 0 rpy=1.57 0 0
- joint laser_joint: child base_laser_link -> laser_link; parent base_link -> real_base_link
- joint neckHead_joint: origin xyz=0 0 0.11 rpy=-1.57 0 0 -> xyz=0 0 0.0927 rpy=-1.57 0 0; type fixed -> revolute
- joint sternoclavicular_joint: origin xyz=0 -0.145 0 rpy=0 -1.57 0 -> xyz=0.008948 -0.145 0.155 rpy=0 -1.57 0
- joint torsoNeck_joint: origin xyz=0 0 0.09 rpy=0 0 0 -> xyz=0.032295 0 0.2437 rpy=0 0 0

Commit message: update urdf

File: sara_description/urdf/sara.urdf (robot description, URDF)
Before this commit: robot sara, 16 links, 15 joints
Links:
- removed link laser_link
- added link base_laser_link, mass 0.5; collision cylinder length=0.1 radius=0.03; visual cylinder length=0.1 radius=0.03
Joints:
- joint laser_joint: child laser_link -> base_laser_link
- joint neckHead_dynamixel_joint: origin xyz=0 -0.054 0 rpy=0 0 0 -> xyz=0 -0.054 0 rpy=3.1416 0 0
