Commit message: Update URDF

File: sara_description/urdf/sara.urdf.xacro (robot description, xacro)
@@ -1,28 +1,29 @@
 <?xml version="1.0"?>
-<robot name="sara">
+<robot xmlns:xacro="http://www.ros.org/wiki/xacro" name="sara">
+    <xacro:include filename="$(find sara_description)/urdf/robotiq_c2_model_macro.xacro" />
 <!-- LINKS -->
-	<link name="base_link">
-		<visual>
-			<geometry>
-				<box size="0.7637 0.64311 0.14" />
-			</geometry>
-			<origin xyz="0.0 0.0 0.07" rpy="0.0 0.0 0.0" />
-		</visual>
-	</link>
-	<link name="base_x_trans_link">
-		<visual>
-			<geometry>
-				<box size="0.10 0.64311 0.14" />
-			</geometry>
-			<origin origin="0.0 0.0 0.07" rpy="0 0 0" />
-		</visual>
-	</link>
-	<link name="base_y_trans_link">
-		<visual>
-			<geometry>
-				<box size="0.7637 0.10 0.14" />
-			</geometry>
-		</visual>
-	</link>
+    <link name="base_link">
+	<visual>
+		<geometry>
+	            <box size="0.7637 0.64311 0.14" />
+		</geometry>
+	    <origin xyz="0.0 0.0 0.07" rpy="0.0 0.0 0.0" />
+	</visual>
+    </link>
+    <link name="base_x_trans_link">
+	<visual>
+		<geometry>
+		    <box size="0.10 0.64311 0.14" />
+		</geometry>
+	    <origin origin="0.0 0.0 0.07" rpy="0 0 0" />
+	</visual>
+    </link>
+    <link name="base_y_trans_link">
+	<visual>
+	    <geometry>
+	        <box size="0.7637 0.10 0.14" />
+	    </geometry>
+	</visual>
+    </link>
     <link name="real_base_link">
         <visual>
@@ -238,5 +239,5 @@
         <visual>
             <geometry>
-                <mesh filename="package://sara_description/meshes/pince-avant-bras.STL" scale="0.001 0.001 0.001"/>
+                <mesh filename="package://sara_description/meshes/avant-bras.STL" scale="0.001 0.001 0.001"/>
             </geometry>
             <origin xyz="0 0 0" rpy="-1.5708 0 -1.5708"/>
@@ -244,41 +245,34 @@
         <collision>
             <geometry>
-                <mesh filename="package://sara_description/meshes/pince-avant-bras.STL" scale="0.001 0.001 0.001"/>
+                <mesh filename="package://sara_description/meshes/avant-bras.STL" scale="0.001 0.001 0.001"/>
             </geometry>
             <origin xyz="0 0 0" rpy="-1.5708 0 -1.5708"/>
         </collision>
     </link>
-    <!--
-    <link name="gripper_link">
-        <visual>
-            <geometry>
-                <cylinder length="0.6" radius="0.1"/>
-            </geometry>
-            <origin xyz="0 0 -0.3" rpy="0 0 0"/>
-        </visual>
-    </link>
-    -->
+    <xacro:robotiq_c2_model prefix="">
+      <origin xyz="0 0 0" rpy="0 0 0" />
+    </xacro:robotiq_c2_model>
   <!-- JOINTS -->
-	<joint name="base_x_trans_joint" type="prismatic" >
-		<parent link="base_link" type="prismatic" />
-		<child link="base_x_trans_link" />
-		<origin xyz="0.0 0.0 0.0" rpy="0.0 0.0 0.0" />
-		<limit effort="1000.0" lower="-0.10" upper="4.0" velocity="1.0"/>
-		<axis xyz="1 0 0" />
-	</joint>
-	<joint name="base_y_trans_joint" type="prismatic" >
-		<parent link="base_x_trans_link" type="prismatic" />
-		<child link="base_y_trans_link" />
-		<origin xyz="0.0 0.0 0.0" rpy="0.0 0.0 0.0" />
-		<limit effort="1000.0" lower="-4.0" upper="4.0" velocity="1.0"/>
-		<axis xyz="0 1 0" />
-	</joint>
-	<joint name="base_revolute_joint" type="revolute" >
-		<parent link="base_y_trans_link" />
-		<child link="real_base_link" />
-		<limit effort="1000.0" lower="-1.5708" upper="1.5708" velocity="0.5"/>
-		<origin xyz="0.0 0.0 0.0" rpy="0.0 0.0 0.0" />
-		<axis xyz="0 0 1" />
-	</joint>
+    <joint name="base_x_trans_joint" type="prismatic" >
+	<parent link="base_link" type="prismatic" />
+	<child link="base_x_trans_link" />
+	<origin xyz="0.0 0.0 0.0" rpy="0.0 0.0 0.0" />
+	<limit effort="1000.0" lower="-0.10" upper="4.0" velocity="1.0"/>
+	<axis xyz="1 0 0" />
+    </joint>
+    <joint name="base_y_trans_joint" type="prismatic" >
+	<parent link="base_x_trans_link" type="prismatic" />
+	<child link="base_y_trans_link" />
+	<origin xyz="0.0 0.0 0.0" rpy="0.0 0.0 0.0" />
+	<limit effort="1000.0" lower="-4.0" upper="4.0" velocity="1.0"/>
+	<axis xyz="0 1 0" />
+    </joint>
+    <joint name="base_revolute_joint" type="revolute" >
+	<parent link="base_y_trans_link" />
+	<child link="real_base_link" />
+	<limit effort="1000.0" lower="-1.5708" upper="1.5708" velocity="0.5"/>
+	<origin xyz="0.0 0.0 0.0" rpy="0.0 0.0 0.0" />
+	<axis xyz="0 0 1" />
+    </joint>
     <joint name="laser_joint" type="fixed">
         <parent link="real_base_link"/>
@@ -331,14 +325,13 @@
         <child link="rotLowerArm_link"/>
         <limit effort="1000.0" lower="-3.1416" upper="3.1416" velocity="0.5"/>
-        <origin xyz="0 0.0945 0" rpy="1.5708 0 0" />
-        <axis xyz="0 0 1" />
-    </joint>
-    <!--
+        <origin xyz="0 0.0945 0" rpy="1.5708 -1.5708 0" />
+        <axis xyz="0 0 1" />
+    </joint>
     <joint name="Wrist_joint" type="fixed">
-        <parent link="rotLowerArm_link"/>
-        <child link="gripper_link"/>
-        <origin xyz="0 0 0.2" rpy="0 0 0" />
-    </joint>
-    -->
+      <parent link="rotLowerArm_link"/>"
+      <child link="robotiq_85_base_link"/>
+      <axis xyz="0 0 1"/>
+      <origin xyz="0 0 -0.10624" rpy="0 1.5708 1.5708"/>
+    </joint>
     <joint name="torsoNeck_joint" type="fixed">  <!-- normaly revolute -->
         <parent link="torso_link"/>
@@ -371,4 +364,19 @@
         <gravity>false</gravity>
     </gazebo>
+    <gazebo reference="base_x_trans_link">
+        <gravity>false</gravity>
+    </gazebo>
+    <gazebo reference="base_y_trans_link">
+        <gravity>false</gravity>
+    </gazebo>
+    <gazebo reference="real_base_link">
+        <gravity>false</gravity>
+    </gazebo>
+    <gazebo reference="spine_link">
+        <gravity>false</gravity>
+    </gazebo>
+    <gazebo reference="neckHead_dynamixel_link">
+        <gravity>false</gravity>
+    </gazebo>
     <gazebo reference="torso_link">
         <gravity>false</gravity>
@@ -378,4 +386,22 @@
     </gazebo>
     <gazebo reference="head_link">
+        <gravity>false</gravity>
+    </gazebo>
+    <gazebo reference="clavicule_link">
+        <gravity>false</gravity>
+    </gazebo>
+    <gazebo reference="fixUpperArm_link">
+        <gravity>false</gravity>
+    </gazebo>
+    <gazebo reference="rotUpperArm_link">
+        <gravity>false</gravity>
+    </gazebo>
+    <gazebo reference="fixLowerArm_link">
+        <gravity>false</gravity>
+    </gazebo>
+    <gazebo reference="rotLowerArm_link">
+        <gravity>false</gravity>
+    </gazebo>
+    <gazebo reference="fixUpperArm_link">
         <gravity>false</gravity>
     </gazebo>

Commit message: replace STL meshes by dae meshes

File: sara_description/urdf/sara.urdf.xacro (robot description, xacro)
@@ -69,5 +69,5 @@
 		<collision>
             <geometry>
-                <cylinder length="0.9" radius="0.04"/>
+                <cylinder length="0.9" radius="0.07"/>
             </geometry>
             <origin xyz="0 0 0.49" rpy="0 0 0"/>
@@ -104,5 +104,5 @@
         <visual>
             <geometry>
-                <mesh filename="package://sara_description/meshes/torse.STL" scale="0.001 0.001 0.001"/>
+                <mesh filename="package://sara_description/meshes/torse.dae" scale="0.001 0.001 0.001"/>
             </geometry>
             <origin xyz="0 0 0" rpy="1.5708 0 1.5708"/>
@@ -113,7 +113,7 @@
         <collision>
             <geometry>
-                <mesh filename="package://sara_description/meshes/torse.STL" scale="0.001 0.001 0.001"/>
-            </geometry>
-            <origin xyz="0.01 0 -0.05" rpy="1.5708 0 1.5708"/>
+                <mesh filename="package://sara_description/meshes/torse.dae" scale="0.001 0.001 0.001"/>
+            </geometry>
+            <origin xyz="0 0 0" rpy="1.5708 0 1.5708"/>
         </collision>
         <inertial>
@@ -137,5 +137,5 @@
         <visual>
             <geometry>
-                <mesh filename="package://sara_description/meshes/tete.STL" scale="0.001 0.001 0.001"/>
+                <mesh filename="package://sara_description/meshes/tete.dae" scale="0.001 0.001 0.001"/>
             </geometry>
             <origin xyz="0 0 0" rpy="1.5708 -1.5708 1.5708"/>
@@ -143,7 +143,7 @@
         <collision>
             <geometry>
-                <sphere radius="0.1"/>
-            </geometry>
-            <origin xyz="0 0 0" rpy="1.5708 0 1.5708"/>
+                <mesh filename="package://sara_description/meshes/tete.dae" scale="0.001 0.001 0.001"/>
+            </geometry>
+            <origin xyz="0 0 0" rpy="1.5708 -1.5708 1.5708"/>
         </collision>
         <inertial>
@@ -156,5 +156,5 @@
          <visual>
              <geometry>
-                 <mesh filename="package://sara_description/meshes/cou.STL" scale="0.001 0.001 0.001"/>
+                 <mesh filename="package://sara_description/meshes/cou.dae" scale="0.001 0.001 0.001"/>
              </geometry>
              <origin xyz="0 0 0" rpy="1.5708 0 1.5708"/>
@@ -169,5 +169,5 @@
         <visual>
             <geometry>
-                <mesh filename="package://sara_description/meshes/xtion.STL" scale="0.001 0.001 0.001"/>
+                <mesh filename="package://sara_description/meshes/xtion.dae" scale="0.001 0.001 0.001"/>
             </geometry>
             <origin xyz="0 0 0" rpy="1.5708 0 1.5708"/>
@@ -183,5 +183,5 @@
          <visual>
              <geometry>
-                 <mesh filename="package://sara_description/meshes/epaule.STL" scale="0.001 0.001 0.001"/>
+                 <mesh filename="package://sara_description/meshes/epaule.dae" scale="0.001 0.001 0.001"/>
              </geometry>
              <origin xyz="0 0 0" rpy="0 3.1416 0"/>
@@ -189,7 +189,7 @@
         <collision>
             <geometry>
-                <mesh filename="package://sara_description/meshes/epaule.STL" scale="0.001 0.001 0.001"/>
-            </geometry>
-             <origin xyz="0 0 0" rpy="0 0 0"/>
+                <mesh filename="package://sara_description/meshes/epaule.dae" scale="0.001 0.001 0.001"/>
+            </geometry>
+             <origin xyz="0 0 0" rpy="0 3.1416 0"/>
         </collision>
     </link>
@@ -197,11 +197,11 @@
          <visual>
             <geometry>
-                <mesh filename="package://sara_description/meshes/epaule.STL" scale="0.001 0.001 0.001"/>
+                <mesh filename="package://sara_description/meshes/epaule.dae" scale="0.001 0.001 0.001"/>
             </geometry>
             <origin xyz="0 0 0" rpy="3.1416 0 1.5708"/>
         </visual>
-        <collision>
-            <geometry>
-                <mesh filename="package://sara_description/meshes/epaule.STL" scale="0.001 0.001 0.001"/>
+	    <collision>
+            <geometry>
+                <mesh filename="package://sara_description/meshes/epaule.dae" scale="0.001 0.001 0.001"/>
             </geometry>
             <origin xyz="0 0 0" rpy="3.1416 0 1.5708"/>
@@ -211,5 +211,5 @@
         <visual>
             <geometry>
-                <mesh filename="package://sara_description/meshes/bras_haut.STL" scale="0.001 0.001 0.001"/>
+                <mesh filename="package://sara_description/meshes/bras_haut.dae" scale="0.001 0.001 0.001"/>
             </geometry>
             <origin xyz="0 0 0" rpy="1.5708 3.1416 3.1416"/>
@@ -217,5 +217,5 @@
         <collision>
             <geometry>
-                <mesh filename="package://sara_description/meshes/bras_haut.STL" scale="0.001 0.001 0.001"/>
+                <mesh filename="package://sara_description/meshes/bras_haut.dae" scale="0.001 0.001 0.001"/>
             </geometry>
             <origin xyz="0 0 0" rpy="1.5708 3.1416 3.1416"/>
@@ -225,5 +225,5 @@
         <visual>
             <geometry>
-                <mesh filename="package://sara_description/meshes/coude.STL" scale="0.001 0.001 0.001"/>
+                <mesh filename="package://sara_description/meshes/coude.dae" scale="0.001 0.001 0.001"/>
             </geometry>
             <origin xyz="0 0 -0.0005" rpy="3.1416 0 0"/>
@@ -231,5 +231,5 @@
         <collision>
              <geometry>
-                <mesh filename="package://sara_description/meshes/coude.STL" scale="0.001 0.001 0.001"/>
+                <mesh filename="package://sara_description/meshes/coude.dae" scale="0.001 0.001 0.001"/>
             </geometry>
             <origin xyz="0 0 -0.0005" rpy="3.1416 0 0"/>
@@ -239,5 +239,5 @@
         <visual>
             <geometry>
-                <mesh filename="package://sara_description/meshes/avant-bras.STL" scale="0.001 0.001 0.001"/>
+                <mesh filename="package://sara_description/meshes/avant-bras.dae" scale="0.001 0.001 0.001"/>
             </geometry>
             <origin xyz="0 0 0" rpy="-1.5708 0 -1.5708"/>
@@ -245,5 +245,5 @@
         <collision>
             <geometry>
-                <mesh filename="package://sara_description/meshes/avant-bras.STL" scale="0.001 0.001 0.001"/>
+                <mesh filename="package://sara_description/meshes/avant-bras.dae" scale="0.001 0.001 0.001"/>
             </geometry>
             <origin xyz="0 0 0" rpy="-1.5708 0 -1.5708"/>
@@ -328,8 +328,9 @@
         <axis xyz="0 0 1" />
     </joint>
-    <joint name="Wrist_joint" type="fixed">
+    <joint name="Wrist_joint" type="revolute"> <!-- normally fixed, dummy revolute joint -->
       <parent link="rotLowerArm_link"/>"
       <child link="robotiq_85_base_link"/>
-      <axis xyz="0 0 1"/>
+	  <limit effort="1000.0" lower="-0.03" upper="0.03" velocity="0.5" />
+      <axis xyz="1 0 0"/>
       <origin xyz="0 0 -0.10624" rpy="0 1.5708 1.5708"/>
     </joint>

Commit message: fix neck/head tf tree

File: sara_description/urdf/sara.urdf.xacro (robot description, xacro)
@@ -128,5 +128,5 @@
                 <cylinder length="0.015" radius="0.02"/>
             </geometry>
-            <origin xyz="0 0 -0.01" rpy="0 0 0"/>
+            <origin xyz="0 0 0" rpy="0 0 0"/>
             <material name="blue">
                 <color rgba="0 0 1 1"/>
@@ -343,15 +343,15 @@
     </joint>
     <joint name="neckHead_dynamixel_joint" type="revolute">
-        <parent link="head_link"/>
+        <parent link="neck_link"/>
         <child link="neckHead_dynamixel_link"/>
         <limit effort="1000.0" lower="-1.5" upper="1.5" velocity="0.5"/>
-        <origin xyz="0 -0.054 0" rpy="3.1416 0 0" />
+        <origin xyz="0 0 0.0927 " rpy="-1.5708 0 0" />
         <axis xyz="0 0 1" />
     </joint>
     <joint name="neckHead_joint" type="revolute">
-        <parent link="neck_link"/>
+        <parent link="neckHead_dynamixel_link"/>
         <child link="head_link"/>
         <limit effort="1000.0" lower="-0.40" upper="1.04" velocity="0.5"/>
-        <origin xyz="0 0 0.0927" rpy="-1.57 0 0" />
+        <origin xyz="0 0 0" rpy="0 0 0" />
         <axis xyz="0 0 1" />
     </joint>

Commit message: removed all the .pyc file + update neck, urdf

File: sara_description/urdf/sara.urdf.xacro (robot description, xacro)
@@ -290,5 +290,5 @@
         <child link="torso_link"/>
         <limit effort="1000.0" lower="0" upper="0.5" velocity="0.2"/>
-        <origin xyz="0 0 1" rpy="0 0 0" />
+        <origin xyz="0 0 1.05" rpy="0 0 0" />
         <axis xyz="0 0 1" />
     </joint>
@@ -342,18 +342,18 @@
         <axis xyz="0 0 1" />
     </joint>
-    <joint name="neckHead_dynamixel_joint" type="revolute">
-        <parent link="neck_link"/>
-        <child link="neckHead_dynamixel_link"/>
-        <limit effort="1000.0" lower="-1.5" upper="1.5" velocity="0.5"/>
-        <origin xyz="0 0 0.0927 " rpy="-1.5708 0 0" />
-        <axis xyz="0 0 1" />
-    </joint>
-    <joint name="neckHead_joint" type="revolute">
-        <parent link="neckHead_dynamixel_link"/>
-        <child link="head_link"/>
-        <limit effort="1000.0" lower="-0.40" upper="1.04" velocity="0.5"/>
-        <origin xyz="0 0 0" rpy="0 0 0" />
-        <axis xyz="0 0 1" />
-    </joint>
+     <joint name="neckHead_dynamixel_joint" type="revolute">
+         <parent link="head_link"/>
+         <child link="neckHead_dynamixel_link"/>
+         <limit effort="1000.0" lower="-1.5" upper="1.5" velocity="0.5"/>
+         <origin xyz="0 -0.054 0" rpy="3.1416 0 0" />
+         <axis xyz="0 0 1" />
+     </joint>
+     <joint name="neckHead_joint" type="revolute">
+         <parent link="neck_link"/>
+         <child link="head_link"/>
+         <limit effort="1000.0" lower="-0.40" upper="1.04" velocity="0.5"/>
+         <origin xyz="0 0 0.0927" rpy="-1.57 0 0" />
+         <axis xyz="0 0 1" />
+     </joint>
     <joint name="camera_joint" type="fixed">
         <parent link="head_link"/>

Commit message: add grip_link

File: sara_description/urdf/sara.urdf.xacro (robot description, xacro)
@@ -253,4 +253,12 @@
       <origin xyz="0 0 0" rpy="0 0 0" />
     </xacro:robotiq_c2_model>
+	<link name="grip_link" >
+		<visual>
+			<geometry>
+				<sphere radius="0.01" />
+			</geometry>
+			<origin xyz="0 0 0" rpy="0 0 0" />
+		</visual>
+	</link>
   <!-- JOINTS -->
     <joint name="base_x_trans_joint" type="prismatic" >
@@ -335,4 +343,9 @@
       <origin xyz="0 0 -0.10624" rpy="0 1.5708 1.5708"/>
     </joint>
+	<joint name="grip_joint" type="fixed" >
+		<parent link="robotiq_85_base_link" />
+		<child link="grip_link" />
+		<origin xyz="0.12 0 -0.012" rpy="3.1416 0 1.5708" />
+	</joint>
     <joint name="torsoNeck_joint" type="fixed">  <!-- normaly revolute -->
         <parent link="torso_link"/>

Commit message: rename grip_link/grip_joint to grasp_link/grasp_joint

File: sara_description/urdf/sara.urdf.xacro (robot description, xacro)
@@ -253,5 +253,5 @@
       <origin xyz="0 0 0" rpy="0 0 0" />
     </xacro:robotiq_c2_model>
-	<link name="grip_link" >
+	<link name="grasp_link" >
 		<visual>
 			<geometry>
@@ -343,7 +343,7 @@
       <origin xyz="0 0 -0.10624" rpy="0 1.5708 1.5708"/>
     </joint>
-	<joint name="grip_joint" type="fixed" >
+	<joint name="grasp_joint" type="fixed" >
 		<parent link="robotiq_85_base_link" />
-		<child link="grip_link" />
+		<child link="grasp_link" />
 		<origin xyz="0.12 0 -0.012" rpy="3.1416 0 1.5708" />
 	</joint>

Commit message: update wrist link dummy joint

File: sara_description/urdf/sara.urdf.xacro (robot description, xacro)
@@ -339,6 +339,6 @@
       <parent link="rotLowerArm_link"/>"
       <child link="robotiq_85_base_link"/>
-	  <limit effort="1000.0" lower="-0.03" upper="0.03" velocity="0.5" />
-      <axis xyz="1 0 0"/>
+	  <limit effort="1000.0" lower="-0.26" upper="0.26" velocity="0.5" />
+      <axis xyz="0 1 0"/>
       <origin xyz="0 0 -0.10624" rpy="0 1.5708 1.5708"/>
     </joint>

Commit message: update torso height

File: sara_description/urdf/sara.urdf.xacro (robot description, xacro)
@@ -298,5 +298,5 @@
         <child link="torso_link"/>
         <limit effort="1000.0" lower="0" upper="0.5" velocity="0.2"/>
-        <origin xyz="0 0 1.05" rpy="0 0 0" />
+        <origin xyz="0 0 1.112" rpy="0 0 0" />
         <axis xyz="0 0 1" />
     </joint>

Commit message: update base prismatic joints limits

File: sara_description/urdf/sara.urdf.xacro (robot description, xacro)
@@ -266,5 +266,5 @@
 	<child link="base_x_trans_link" />
 	<origin xyz="0.0 0.0 0.0" rpy="0.0 0.0 0.0" />
-	<limit effort="1000.0" lower="-0.10" upper="4.0" velocity="1.0"/>
+	<limit effort="1000.0" lower="-0.10" upper="1.5" velocity="1.0"/>
 	<axis xyz="1 0 0" />
     </joint>
@@ -273,5 +273,5 @@
 	<child link="base_y_trans_link" />
 	<origin xyz="0.0 0.0 0.0" rpy="0.0 0.0 0.0" />
-	<limit effort="1000.0" lower="-4.0" upper="4.0" velocity="1.0"/>
+	<limit effort="1000.0" lower="-1.5" upper="1.5" velocity="1.0"/>
 	<axis xyz="0 1 0" />
     </joint>

Commit message: remove visual from grasp_link

File: sara_description/urdf/sara.urdf.xacro (robot description, xacro)
@@ -253,12 +253,5 @@
       <origin xyz="0 0 0" rpy="0 0 0" />
     </xacro:robotiq_c2_model>
-	<link name="grasp_link" >
-		<visual>
-			<geometry>
-				<sphere radius="0.01" />
-			</geometry>
-			<origin xyz="0 0 0" rpy="0 0 0" />
-		</visual>
-	</link>
+	<link name="grasp_link" />
   <!-- JOINTS -->
     <joint name="base_x_trans_joint" type="prismatic" >

Commit message: update grasp_link position

File: sara_description/urdf/sara.urdf.xacro (robot description, xacro)
@@ -253,5 +253,12 @@
       <origin xyz="0 0 0" rpy="0 0 0" />
     </xacro:robotiq_c2_model>
-	<link name="grasp_link" />
+	<link name="grasp_link" >
+		<visual>
+			<geometry>
+				<sphere radius="0.01" />
+			</geometry>
+			<origin xyz="0 0 0" rpy="0 0 0" />
+		</visual>
+	</link>
   <!-- JOINTS -->
     <joint name="base_x_trans_joint" type="prismatic" >
@@ -339,5 +346,5 @@
 		<parent link="robotiq_85_base_link" />
 		<child link="grasp_link" />
-		<origin xyz="0.12 0 -0.012" rpy="3.1416 0 1.5708" />
+		<origin xyz="0.075 0 -0.012" rpy="3.1416 0 1.5708" />
 	</joint>
     <joint name="torsoNeck_joint" type="fixed">  <!-- normaly revolute -->

Commit message: update base joint limits

File: sara_description/urdf/sara.urdf.xacro (robot description, xacro)
@@ -263,23 +263,23 @@
   <!-- JOINTS -->
     <joint name="base_x_trans_joint" type="prismatic" >
-	<parent link="base_link" type="prismatic" />
-	<child link="base_x_trans_link" />
-	<origin xyz="0.0 0.0 0.0" rpy="0.0 0.0 0.0" />
-	<limit effort="1000.0" lower="-0.10" upper="1.5" velocity="1.0"/>
-	<axis xyz="1 0 0" />
+		<parent link="base_link" type="prismatic" />
+		<child link="base_x_trans_link" />
+		<origin xyz="0.0 0.0 0.0" rpy="0.0 0.0 0.0" />
+		<limit effort="1000.0" lower="-0.40" upper="1.0" velocity="1.0"/>
+		<axis xyz="1 0 0" />
     </joint>
     <joint name="base_y_trans_joint" type="prismatic" >
-	<parent link="base_x_trans_link" type="prismatic" />
-	<child link="base_y_trans_link" />
-	<origin xyz="0.0 0.0 0.0" rpy="0.0 0.0 0.0" />
-	<limit effort="1000.0" lower="-1.5" upper="1.5" velocity="1.0"/>
-	<axis xyz="0 1 0" />
+		<parent link="base_x_trans_link" type="prismatic" />
+		<child link="base_y_trans_link" />
+		<origin xyz="0.0 0.0 0.0" rpy="0.0 0.0 0.0" />
+		<limit effort="1000.0" lower="-1.0" upper="1.0" velocity="1.0"/>
+		<axis xyz="0 1 0" />
     </joint>
     <joint name="base_revolute_joint" type="revolute" >
-	<parent link="base_y_trans_link" />
-	<child link="real_base_link" />
-	<limit effort="1000.0" lower="-1.5708" upper="1.5708" velocity="0.5"/>
-	<origin xyz="0.0 0.0 0.0" rpy="0.0 0.0 0.0" />
-	<axis xyz="0 0 1" />
+		<parent link="base_y_trans_link" />
+		<child link="real_base_link" />
+		<limit effort="1000.0" lower="-1.5708" upper="1.5708" velocity="0.5"/>
+		<origin xyz="0.0 0.0 0.0" rpy="0.0 0.0 0.0" />
+		<axis xyz="0 0 1" />
     </joint>
     <joint name="laser_joint" type="fixed">
