Commit message: blabla

File: sara_description/urdf/sara.urdf.xacro (robot description, xacro)
@@ -266,5 +266,5 @@
 		<child link="base_x_trans_link" />
 		<origin xyz="0.0 0.0 0.0" rpy="0.0 0.0 0.0" />
-		<limit effort="1000.0" lower="-0.40" upper="1.0" velocity="1.0"/>
+		<limit effort="1000.0" lower="-0.20" upper="0.2" velocity="1.0"/>
 		<axis xyz="1 0 0" />
     </joint>
@@ -273,5 +273,5 @@
 		<child link="base_y_trans_link" />
 		<origin xyz="0.0 0.0 0.0" rpy="0.0 0.0 0.0" />
-		<limit effort="1000.0" lower="-1.0" upper="1.0" velocity="1.0"/>
+		<limit effort="1000.0" lower="-0.4" upper="0.4" velocity="1.0"/>
 		<axis xyz="0 1 0" />
     </joint>

Commit message: Update URDF with new format

File: sara_description/urdf/sara.urdf.xacro (robot description, xacro)
@@ -1,507 +1,16 @@
 <?xml version="1.0"?>
-<robot xmlns:xacro="http://www.ros.org/wiki/xacro" name="sara">
-    <xacro:include filename="$(find sara_description)/urdf/robotiq_c2_model_macro.xacro" />
-<!-- LINKS -->
-    <link name="base_link">
-	<visual>
-		<geometry>
-	            <box size="0.7637 0.64311 0.14" />
-		</geometry>
-	    <origin xyz="0.0 0.0 0.07" rpy="0.0 0.0 0.0" />
-	</visual>
-    </link>
-    <link name="base_x_trans_link">
-	<visual>
-		<geometry>
-		    <box size="0.10 0.64311 0.14" />
-		</geometry>
-	    <origin origin="0.0 0.0 0.07" rpy="0 0 0" />
-	</visual>
-    </link>
-    <link name="base_y_trans_link">
-	<visual>
-	    <geometry>
-	        <box size="0.7637 0.10 0.14" />
-	    </geometry>
-	</visual>
-    </link>
-    <link name="real_base_link">
-        <visual>
-            <geometry>
-                <box size="0.7637 0.64311 0.14"/>
-            </geometry>
-            <origin xyz="0.0 0 0.07" rpy="0 0 0"/>
-            <material name="grey">
-                <color rgba="0.62 0.62 0.62 1"/>
-            </material>
-        </visual>
-        <visual>
-            <geometry>
-                <box size="0.55 0.64311 0.57"/>
-            </geometry>
-            <origin xyz="-0.115 0 0.42" rpy="0 0 0"/>
-        </visual>
-        <collision>
-            <geometry>
-                <box size="0.7637 0.64311 0.14"/>
-            </geometry>
-            <origin xyz="0.0 0 0.07" rpy="0 0 0"/>
-        </collision>
-        <collision>
-            <geometry>
-                <box size="0.55 0.64311 0.57"/>
-            </geometry>
-            <origin xyz="-0.115 0 0.42" rpy="0 0 0"/>
-        </collision>
-        <inertial>
-            <mass value="10"/>
-            <origin xyz="-0.115 0 0.42" rpy="0 0 0"/>
-            <inertia ixx="0.001" ixy="0" ixz="0" iyy="0.001" iyz="0" izz="0.001"/>
-        </inertial>
-    </link>
-    <link name="spine_link">
-        <visual>
-            <geometry>
-                <cylinder length="0.9" radius="0.04"/>
-            </geometry>
-            <origin xyz="0 0 0.49" rpy="0 0 0"/>
-        </visual>
-		<collision>
-            <geometry>
-                <cylinder length="0.9" radius="0.07"/>
-            </geometry>
-            <origin xyz="0 0 0.49" rpy="0 0 0"/>
-        </collision>
-        <inertial>
-            <mass value="10"/>
-            <origin xyz="0 0 0.49" rpy="0 0 0"/>
-            <inertia ixx="0.001" ixy="0" ixz="0" iyy="0.001" iyz="0" izz="0.001"/>
-        </inertial>
-    </link>
-    <link name="base_laser_link">
-        <visual>
-            <geometry>
-                <cylinder length="0.1" radius="0.03"/>
-            </geometry>
-            <origin xyz="0 0 0" rpy="0 0 0"/>
-            <material name="orange">
-                <color rgba="1 0.5 0 1"/>
-            </material>
-        </visual>
-        <collision>
-            <geometry>
-                <cylinder length="0.1" radius="0.03"/>
-            </geometry>
-            <origin xyz="0 0 0" rpy="0 0 0"/>
-        </collision>
-        <inertial>
-            <mass value="0.5"/>
-            <origin xyz="0 0 0" rpy="0 0 0"/>
-            <inertia ixx="0.001" ixy="0" ixz="0" iyy="0.001" iyz="0" izz="0.001"/>
-        </inertial>
-    </link>
-    <link name="torso_link">
-        <visual>
-            <geometry>
-                <mesh filename="package://sara_description/meshes/torse.dae" scale="0.001 0.001 0.001"/>
-            </geometry>
-            <origin xyz="0 0 0" rpy="1.5708 0 1.5708"/>
-            <material name="black">
-                <color rgba="0.12 0.12 0.12 1"/>
-            </material>
-        </visual>
-        <collision>
-            <geometry>
-                <mesh filename="package://sara_description/meshes/torse.dae" scale="0.001 0.001 0.001"/>
-            </geometry>
-            <origin xyz="0 0 0" rpy="1.5708 0 1.5708"/>
-        </collision>
-        <inertial>
-            <mass value="10"/>
-            <origin xyz="0 0 0" rpy="1.5708 0 1.5708"/>
-            <inertia ixx="0.001" ixy="0" ixz="0" iyy="0.001" iyz="0" izz="0.001"/>
-        </inertial>
-    </link>
-    <link name="neckHead_dynamixel_link">
-        <visual>
-            <geometry>
-                <cylinder length="0.015" radius="0.02"/>
-            </geometry>
-            <origin xyz="0 0 0" rpy="0 0 0"/>
-            <material name="blue">
-                <color rgba="0 0 1 1"/>
-            </material>
-        </visual>
-    </link>
-    <link name="head_link">
-        <visual>
-            <geometry>
-                <mesh filename="package://sara_description/meshes/tete.dae" scale="0.001 0.001 0.001"/>
-            </geometry>
-            <origin xyz="0 0 0" rpy="1.5708 -1.5708 1.5708"/>
-        </visual>
-        <collision>
-            <geometry>
-                <mesh filename="package://sara_description/meshes/tete.dae" scale="0.001 0.001 0.001"/>
-            </geometry>
-            <origin xyz="0 0 0" rpy="1.5708 -1.5708 1.5708"/>
-        </collision>
-        <inertial>
-            <mass value="5"/>
-            <origin xyz="0 0 0" rpy="1.5708 0 1.5708"/>
-            <inertia ixx="0.001" ixy="0" ixz="0" iyy="0.001" iyz="0" izz="0.001"/>
-        </inertial>
-    </link>
-    <link name="neck_link">
-         <visual>
-             <geometry>
-                 <mesh filename="package://sara_description/meshes/cou.dae" scale="0.001 0.001 0.001"/>
-             </geometry>
-             <origin xyz="0 0 0" rpy="1.5708 0 1.5708"/>
-        </visual>
-        <inertial>
-            <mass value="2"/>
-            <origin xyz="0 0 0" rpy="1.5708 0 1.5708"/>
-            <inertia ixx="0.001" ixy="0" ixz="0" iyy="0.001" iyz="0" izz="0.001"/>
-        </inertial>
-    </link>
-    <link name="camera_link">
-        <visual>
-            <geometry>
-                <mesh filename="package://sara_description/meshes/xtion.dae" scale="0.001 0.001 0.001"/>
-            </geometry>
-            <origin xyz="0 0 0" rpy="1.5708 0 1.5708"/>
-            <material name="black"/>
-        </visual>
-        <inertial>
-            <mass value="0.5"/>
-            <origin xyz="0 0 0" rpy="1.5708 0 1.5708"/>
-            <inertia ixx="0.001" ixy="0" ixz="0" iyy="0.001" iyz="0" izz="0.001"/>
-        </inertial>
-    </link>
-    <link name="clavicule_link">
-         <visual>
-             <geometry>
-                 <mesh filename="package://sara_description/meshes/epaule.dae" scale="0.001 0.001 0.001"/>
-             </geometry>
-             <origin xyz="0 0 0" rpy="0 3.1416 0"/>
-         </visual>
-        <collision>
-            <geometry>
-                <mesh filename="package://sara_description/meshes/epaule.dae" scale="0.001 0.001 0.001"/>
-            </geometry>
-             <origin xyz="0 0 0" rpy="0 3.1416 0"/>
-        </collision>
-    </link>
-    <link name="fixUpperArm_link">
-         <visual>
-            <geometry>
-                <mesh filename="package://sara_description/meshes/epaule.dae" scale="0.001 0.001 0.001"/>
-            </geometry>
-            <origin xyz="0 0 0" rpy="3.1416 0 1.5708"/>
-        </visual>
-	    <collision>
-            <geometry>
-                <mesh filename="package://sara_description/meshes/epaule.dae" scale="0.001 0.001 0.001"/>
-            </geometry>
-            <origin xyz="0 0 0" rpy="3.1416 0 1.5708"/>
-        </collision>
-    </link>
-    <link name="rotUpperArm_link">
-        <visual>
-            <geometry>
-                <mesh filename="package://sara_description/meshes/bras_haut.dae" scale="0.001 0.001 0.001"/>
-            </geometry>
-            <origin xyz="0 0 0" rpy="1.5708 3.1416 3.1416"/>
-        </visual>
-        <collision>
-            <geometry>
-                <mesh filename="package://sara_description/meshes/bras_haut.dae" scale="0.001 0.001 0.001"/>
-            </geometry>
-            <origin xyz="0 0 0" rpy="1.5708 3.1416 3.1416"/>
-        </collision>
-    </link>
-    <link name="fixLowerArm_link">
-        <visual>
-            <geometry>
-                <mesh filename="package://sara_description/meshes/coude.dae" scale="0.001 0.001 0.001"/>
-            </geometry>
-            <origin xyz="0 0 -0.0005" rpy="3.1416 0 0"/>
-        </visual>
-        <collision>
-             <geometry>
-                <mesh filename="package://sara_description/meshes/coude.dae" scale="0.001 0.001 0.001"/>
-            </geometry>
-            <origin xyz="0 0 -0.0005" rpy="3.1416 0 0"/>
-        </collision>
-    </link>
-    <link name="rotLowerArm_link">
-        <visual>
-            <geometry>
-                <mesh filename="package://sara_description/meshes/avant-bras.dae" scale="0.001 0.001 0.001"/>
-            </geometry>
-            <origin xyz="0 0 0" rpy="-1.5708 0 -1.5708"/>
-        </visual>
-        <collision>
-            <geometry>
-                <mesh filename="package://sara_description/meshes/avant-bras.dae" scale="0.001 0.001 0.001"/>
-            </geometry>
-            <origin xyz="0 0 0" rpy="-1.5708 0 -1.5708"/>
-        </collision>
-    </link>
-    <xacro:robotiq_c2_model prefix="">
-      <origin xyz="0 0 0" rpy="0 0 0" />
-    </xacro:robotiq_c2_model>
-	<link name="grasp_link" >
-		<visual>
-			<geometry>
-				<sphere radius="0.01" />
-			</geometry>
-			<origin xyz="0 0 0" rpy="0 0 0" />
-		</visual>
-	</link>
-  <!-- JOINTS -->
-    <joint name="base_x_trans_joint" type="prismatic" >
-		<parent link="base_link" type="prismatic" />
-		<child link="base_x_trans_link" />
-		<origin xyz="0.0 0.0 0.0" rpy="0.0 0.0 0.0" />
-		<limit effort="1000.0" lower="-0.20" upper="0.2" velocity="1.0"/>
-		<axis xyz="1 0 0" />
-    </joint>
-    <joint name="base_y_trans_joint" type="prismatic" >
-		<parent link="base_x_trans_link" type="prismatic" />
-		<child link="base_y_trans_link" />
-		<origin xyz="0.0 0.0 0.0" rpy="0.0 0.0 0.0" />
-		<limit effort="1000.0" lower="-0.4" upper="0.4" velocity="1.0"/>
-		<axis xyz="0 1 0" />
-    </joint>
-    <joint name="base_revolute_joint" type="revolute" >
-		<parent link="base_y_trans_link" />
-		<child link="real_base_link" />
-		<limit effort="1000.0" lower="-1.5708" upper="1.5708" velocity="0.5"/>
-		<origin xyz="0.0 0.0 0.0" rpy="0.0 0.0 0.0" />
-		<axis xyz="0 0 1" />
-    </joint>
-    <joint name="laser_joint" type="fixed">
-        <parent link="real_base_link"/>
-        <child link="base_laser_link"/>
-        <origin xyz="0.34 0 0.19" rpy="0 0 0" />
-    </joint>
-    <joint name="base_spine_joint" type="fixed">
-        <parent link="real_base_link"/>
-        <child link="spine_link"/>
-        <origin xyz="0.2 0 0" rpy="0 0 0" />
-        <axis xyz="0 0 1" />
-    </joint>
-    <joint name="spine_torso_joint" type="fixed"> <!-- normaly prismatic -->
-        <parent link="spine_link"/>
-        <child link="torso_link"/>
-        <limit effort="1000.0" lower="0" upper="0.5" velocity="0.2"/>
-        <origin xyz="0 0 1.112" rpy="0 0 0" />
-        <axis xyz="0 0 1" />
-    </joint>
-    <joint name="sternoclavicular_joint" type="revolute">
-        <parent link="torso_link"/>
-        <child link="clavicule_link"/>
-        <limit effort="1000.0" lower="-0.18" upper="1.21" velocity="0.5"/>
-        <origin xyz="0.008948 -0.145 0.155" rpy="0 -1.57 0" />
-        <axis xyz="0 0 1" />
-    </joint>
-    <joint name="shoulder_joint" type="revolute">
-        <parent link="clavicule_link"/>
-        <child link="fixUpperArm_link"/>
-        <limit effort="1000.0" lower="-3.29" upper="0.37" velocity="0.5"/>
-        <origin xyz="0 -0.085 0" rpy="-1.57 0 0" />
-        <axis xyz="0 0 1" />
-    </joint>
-    <joint name="shoulderRot_joint" type="revolute">
-        <parent link="fixUpperArm_link"/>
-        <child link="rotUpperArm_link"/>
-        <limit effort="1000.0" lower="-2.14" upper="1.00" velocity="0.5"/>
-        <origin xyz="-0.085 0 0" rpy="1.5708 0 1.5708" />
-        <axis xyz="0 0 1" />
-    </joint>
-    <joint name="elbow_joint" type="revolute">
-        <parent link="rotUpperArm_link"/>
-        <child link="fixLowerArm_link"/>
-        <limit effort="1000.0" lower="-2.20" upper="1.90" velocity="0.5"/>
-        <origin xyz="0 0 -0.31" rpy="-1.5708 0 0" />
-        <axis xyz="0 0 1" />
-    </joint>
-    <joint name="WristRot_joint" type="revolute">
-        <parent link="fixLowerArm_link"/>
-        <child link="rotLowerArm_link"/>
-        <limit effort="1000.0" lower="-3.1416" upper="3.1416" velocity="0.5"/>
-        <origin xyz="0 0.0945 0" rpy="1.5708 -1.5708 0" />
-        <axis xyz="0 0 1" />
-    </joint>
-    <joint name="Wrist_joint" type="revolute"> <!-- normally fixed, dummy revolute joint -->
-      <parent link="rotLowerArm_link"/>"
-      <child link="robotiq_85_base_link"/>
-	  <limit effort="1000.0" lower="-0.26" upper="0.26" velocity="0.5" />
-      <axis xyz="0 1 0"/>
-      <origin xyz="0 0 -0.10624" rpy="0 1.5708 1.5708"/>
-    </joint>
-	<joint name="grasp_joint" type="fixed" >
-		<parent link="robotiq_85_base_link" />
-		<child link="grasp_link" />
-		<origin xyz="0.075 0 -0.012" rpy="3.1416 0 1.5708" />
-	</joint>
-    <joint name="torsoNeck_joint" type="fixed">  <!-- normaly revolute -->
-        <parent link="torso_link"/>
-        <child link="neck_link"/>
-        <limit effort="1000.0" lower="-3.1416" upper="3.1416" velocity="0.5"/>
-        <origin xyz="0.032295 0 0.2437" rpy="0 0 0" />
-        <axis xyz="0 0 1" />
-    </joint>
-     <joint name="neckHead_dynamixel_joint" type="revolute">
-         <parent link="head_link"/>
-         <child link="neckHead_dynamixel_link"/>
-         <limit effort="1000.0" lower="-1.5" upper="1.5" velocity="0.5"/>
-         <origin xyz="0 -0.054 0" rpy="3.1416 0 0" />
-         <axis xyz="0 0 1" />
-     </joint>
-     <joint name="neckHead_joint" type="revolute">
-         <parent link="neck_link"/>
-         <child link="head_link"/>
-         <limit effort="1000.0" lower="-0.40" upper="1.04" velocity="0.5"/>
-         <origin xyz="0 0 0.0927" rpy="-1.57 0 0" />
-         <axis xyz="0 0 1" />
-     </joint>
-    <joint name="camera_joint" type="fixed">
-        <parent link="head_link"/>
-        <child link="camera_link"/>
-        <origin xyz="0.0776104 -0.13 0" rpy="1.57 0 0" />
-        <axis xyz="0 1 0" />
-    </joint>
-    <gazebo reference="base_link">
-        <gravity>false</gravity>
-    </gazebo>
-    <gazebo reference="base_x_trans_link">
-        <gravity>false</gravity>
-    </gazebo>
-    <gazebo reference="base_y_trans_link">
-        <gravity>false</gravity>
-    </gazebo>
-    <gazebo reference="real_base_link">
-        <gravity>false</gravity>
-    </gazebo>
-    <gazebo reference="spine_link">
-        <gravity>false</gravity>
-    </gazebo>
-    <gazebo reference="neckHead_dynamixel_link">
-        <gravity>false</gravity>
-    </gazebo>
-    <gazebo reference="torso_link">
-        <gravity>false</gravity>
-    </gazebo>
-    <gazebo reference="neck_link">
-        <gravity>false</gravity>
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
Commit message: WIP Ajout de la kinect dans le urdf

File: sara_description/urdf/sara.urdf.xacro (robot description, xacro)
@@ -166,5 +166,18 @@
         </inertial>
     </link>
-    <link name="camera_link">
+    <link name="kinect_link">
+        <visual>
+            <geometry>
+                <box size="0.02 0.1 0.01"/>
+            </geometry>            <origin xyz="0 0 0" rpy="1.5708 0 1.5708"/>
+            <material name="black"/>
+        </visual>
+        <inertial>
+            <mass value="0.5"/>
+            <origin xyz="0 0 0" rpy="1.5708 0 1.5708"/>
+            <inertia ixx="0.001" ixy="0" ixz="0" iyy="0.001" iyz="0" izz="0.001"/>
+        </inertial>
+    </link>
+    <link name="xtion_link">
         <visual>
             <geometry>
@@ -301,4 +314,11 @@
         <axis xyz="0 0 1" />
     </joint>
+    <joint name="kinect_joint" type="fixed">
+        <parent link="spine_link"/>
+        <child link="kinect_link"/>
+        <limit effort="1000.0" lower="0" upper="0.5" velocity="0.2"/>
+        <origin xyz="0.156 0 0.165" rpy="0 0 0" />
+        <axis xyz="0 0 1" />
+    </joint>
     <joint name="sternoclavicular_joint" type="revolute">
         <parent link="torso_link"/>
@@ -337,15 +357,15 @@
     </joint>
     <joint name="Wrist_joint" type="revolute"> <!-- normally fixed, dummy revolute joint -->
-      <parent link="rotLowerArm_link"/>"
-      <child link="robotiq_85_base_link"/>
-	  <limit effort="1000.0" lower="-0.26" upper="0.26" velocity="0.5" />
-      <axis xyz="0 1 0"/>
-      <origin xyz="0 0 -0.10624" rpy="0 1.5708 1.5708"/>
-    </joint>
-	<joint name="grasp_joint" type="fixed" >
-		<parent link="robotiq_85_base_link" />
-		<child link="grasp_link" />
-		<origin xyz="0.075 0 -0.012" rpy="3.1416 0 1.5708" />
-	</joint>
+        <parent link="rotLowerArm_link"/>"
+        <child link="robotiq_85_base_link"/>
+	<limit effort="1000.0" lower="-0.26" upper="0.26" velocity="0.5" />
+        <axis xyz="0 1 0"/>
+        <origin xyz="0 0 -0.10624" rpy="0 1.5708 1.5708"/>
+    </joint>
+    <joint name="grasp_joint" type="fixed" >
+	<parent link="robotiq_85_base_link" />
+	<child link="grasp_link" />
+	<origin xyz="0.075 0 -0.012" rpy="3.1416 0 1.5708" />
+    </joint>
     <joint name="torsoNeck_joint" type="fixed">  <!-- normaly revolute -->
         <parent link="torso_link"/>
@@ -369,7 +389,7 @@
          <axis xyz="0 0 1" />
      </joint>
-    <joint name="camera_joint" type="fixed">
+    <joint name="xtion_joint" type="fixed">
         <parent link="head_link"/>
-        <child link="camera_link"/>
+        <child link="xtion_link"/>
         <origin xyz="0.0776104 -0.13 0" rpy="1.57 0 0" />
         <axis xyz="0 1 0" />

Commit message: Fixed wheels xacro macro fail

File: sara_description/urdf/sara.urdf.xacro (robot description, xacro)
@@ -5,5 +5,5 @@
     <xacro:include filename="$(find sara_description)/urdf/neck_v1/neck.urdf.xacro"/>
     <xacro:include filename="$(find sara_description)/urdf/head_v1/head.urdf.xacro"/>
-    <xacro:include filename="$(find sara_description)/urdf/grasp_v1/robotiq_c2_model_macro.xacro"/>
+    <xacro:include filename="$(find sara_description)/urdf/robotiq_c2_model/robotiq_c2_model_macro.xacro"/>
     <xacro:include filename="$(find sara_description)/urdf/arm_v1/arm.urdf.xacro"/>
     <xacro:include filename="$(find sara_description)/urdf/base_v1/base.urdf.xacro"/>
@@ -22,4 +22,4 @@
     <xacro:sara_arm_v1 name="arm" parent="torso" end_effector="robotiq_85_base"/>
     <!-- End Effector -->
-    <xacro:sara_grasp_v1 prefix=""/>
+    <xacro:robotiq_c2_model prefix=""/>
 </robot>

File: sara_description/urdf/wheels_v1/wheels.urdf.xacro (robot description, xacro)
@@ -2,5 +2,6 @@
 <robot xmlns:xacro="http://ros.org/wiki/xacro" >
    <xacro:include filename="$(find sara_description)/urdf/wheels_v1/wheels.gazebo.xacro" />
-   <!-- Front_Wheels -->
+  <xacro:macro name="sara_wheels_v1" params="name parent" >
+  <!-- Front_Wheels -->
   <xacro:macro name="front_wheel" params="prefix y_reflect x_reflect x_axis_rotation">
       <link name="${prefix}_wheel">
@@ -58,3 +59,4 @@
    <xacro:rear_wheel prefix="rear_left" y_reflect="-1" x_reflect="1" x_axis_rotation="-1"/>
    <xacro:rear_wheel prefix="rear_right" y_reflect="-1" x_reflect="-1" x_axis_rotation="1"/>
+ </xacro:macro>
 </robot>
