Commit message: Added torso to new format URDF

File: sara_description/urdf/head_v1/head.urdf.xacro (robot description, xacro)
@@ -39,6 +39,6 @@
          <axis xyz="0 0 1"/>
       </joint>
-      <joint name="dynamixel_${parent}_joint" type="fixed">
-         <parent link="neck_link"/>
+      <joint name="dynamixel_neck_joint" type="fixed">
+         <parent link="${parent}"/>
          <child link="neck_dynamixel_link"/>
          <origin xyz="0 0 0.0927" rpy="1.57 0 0"/>

File: sara_description/urdf/neck_v1/neck.urdf.xacro (robot description, xacro)
@@ -15,4 +15,13 @@
             </inertial>
         </link>
+        <joint name="torso_${name}_joint" type="revolute">
+            <!-- soon revolute -->
+            <parent link="${parent}"/>
+            <child link="${name}_link"/>
+            <limit effort="1000.0" lower="-1.22173" upper="1.22173" velocity="0.5"/>
+            <!-- 1mm ajoute en z (collision) -->
+            <origin xyz="0.032295 0 0.2438" rpy="0 0 0"/>
+            <axis xyz="0 0 1"/>
+        </joint>
     </xacro:macro>
 </robot>

File: sara_description/urdf/sara.urdf.xacro (robot description, xacro)
@@ -4,6 +4,12 @@
     <xacro:include filename="$(find sara_description)/urdf/head_v1/head.urdf.xacro" />
     <xacro:include filename="$(find sara_description)/urdf/neck_v1/neck.urdf.xacro" />
+    <xacro:include filename="$(find sara_description)/urdf/torso_v1/torso.urdf.xacro" />
+    <!-- Torso -->
+    <xacro:sara_torso_v1 name="torso" parent="">
+        <origin xyz="0 0 0"
+                rpy="1.5708 0 1.5708"/>
+    </xacro:sara_torso_v1>
     <!-- Neck -->
-    <xacro:sara_neck_v1 name="neck" parent="">
+    <xacro:sara_neck_v1 name="neck" parent="torso_link">
     	<origin xyz="0 0 0"
     		    rpy="1.5708 0 1.5708"/>

Commit message: Ajout du bras au URDF

File: sara_description/urdf/head_v1/head.urdf.xacro (robot description, xacro)
@@ -40,5 +40,5 @@
       </joint>
       <joint name="dynamixel_neck_joint" type="fixed">
-         <parent link="${parent}"/>
+         <parent link="${parent}_link"/>
          <child link="neck_dynamixel_link"/>
          <origin xyz="0 0 0.0927" rpy="1.57 0 0"/>

File: sara_description/urdf/neck_v1/neck.urdf.xacro (robot description, xacro)
@@ -15,7 +15,6 @@
             </inertial>
         </link>
-        <joint name="torso_${name}_joint" type="revolute">
-            <!-- soon revolute -->
-            <parent link="${parent}"/>
+        <joint name="${parent}_${name}_joint" type="revolute">
+            <parent link="${parent}_link"/>
             <child link="${name}_link"/>
             <limit effort="1000.0" lower="-1.22173" upper="1.22173" velocity="0.5"/>

File: sara_description/urdf/robotiq_c2_model_macro.xacro (robot description, xacro)
@@ -11,5 +11,5 @@
     <visual>
       <geometry>
-        <mesh filename="package://robotiq_c2_model_visualization/meshes/robotiq_c2/visual/robotiq_85_gripper_base.dae"/>
+        <mesh filename="package://sara_description/meshes/robotiq_c2/visual/robotiq_85_gripper_base.dae"/>
       </geometry>
       <origin rpy="3.1415 0 1.5707" xyz="0 0 0"/>
@@ -17,10 +17,9 @@
     <collision>
       <geometry>
-        <mesh filename="package://robotiq_c2_model_visualization/meshes/robotiq_c2/collision/robotiq_85_gripper_base.dae"/>
+        <mesh filename="package://sara_description/meshes/robotiq_c2/collision/robotiq_85_gripper_base.dae"/>
       </geometry>
       <origin rpy="1.5707 0 1.5707" xyz="0 0 0"/>
     </collision>
   </link>
-  <!--  /\  -->
   <joint name="${prefix}robotiq_85_left_knuckle_joint" type="revolute">
     <parent link="${prefix}robotiq_85_base_link"/>
@@ -38,5 +37,4 @@
     <mimic joint="${prefix}robotiq_85_left_knuckle_joint" multiplier="1"/>
   </joint>
-  <!--  \/  -->
   <link name="${prefix}robotiq_85_left_knuckle_link">
     <visual>
@@ -67,6 +65,4 @@
     </collision>
   </link>
-  <!--  /\  -->
-  <!--  /\  -->
   <joint name="${prefix}robotiq_85_left_finger_joint" type="fixed">
     <parent link="${prefix}robotiq_85_left_knuckle_link"/>
@@ -83,6 +79,4 @@
     <limit lower="0" upper="1.5707" velocity="2.0" effort="1000"/>
   </joint>
-  <!--  \/  -->
-  <!--  \/  -->
   <link name="${prefix}robotiq_85_left_finger_link">
     <visual>
@@ -113,6 +107,4 @@
     </collision>
   </link>
-  <!--  /\  -->
-  <!--  /\  -->
   <joint name="${prefix}robotiq_85_left_inner_knuckle_joint" type="revolute">
     <parent link="${prefix}robotiq_85_base_link"/>
@@ -131,6 +123,4 @@
     <mimic joint="${prefix}robotiq_85_left_knuckle_joint" offset="0"/>
   </joint>
-  <!--  \/  -->
-  <!--  \/  -->
   <link name="${prefix}robotiq_85_left_inner_knuckle_link">
     <visual>
@@ -161,6 +151,4 @@
     </collision>
   </link>
-  <!--  /\  -->
-  <!--  /\  -->
   <joint name="${prefix}robotiq_85_left_finger_tip_joint" type="revolute">
     <parent link="${prefix}robotiq_85_left_inner_knuckle_link"/>
@@ -179,6 +167,4 @@
     <mimic joint="${prefix}robotiq_85_left_knuckle_joint" multiplier="-1"/>
   </joint>
-  <!--  \/  -->
-  <!--  \/  -->
   <link name="${prefix}robotiq_85_left_finger_tip_link">
     <visual>

File: sara_description/urdf/sara.urdf.xacro (robot description, xacro)
@@ -2,7 +2,9 @@
 <robot xmlns:xacro="http://playerstage.sourceforge.net/gazebo/xmlschema/#interface" name="sara" >
     <!-- Inclure tous les autres urdf.xacros ici -->
+    <xacro:include filename="$(find sara_description)/urdf/torso_v1/torso.urdf.xacro" />
+    <xacro:include filename="$(find sara_description)/urdf/neck_v1/neck.urdf.xacro" />
     <xacro:include filename="$(find sara_description)/urdf/head_v1/head.urdf.xacro" />
-    <xacro:include filename="$(find sara_description)/urdf/neck_v1/neck.urdf.xacro" />
-    <xacro:include filename="$(find sara_description)/urdf/torso_v1/torso.urdf.xacro" />
+    <xacro:include filename="$(find sara_description)/urdf/shoulder_v1/shoulder.urdf.xacro" />
+    <xacro:include filename="$(find sara_description)/urdf/arm_v1/arm.urdf.xacro" />
     <!-- Torso -->
     <xacro:sara_torso_v1 name="torso" parent="">
@@ -11,12 +13,20 @@
     </xacro:sara_torso_v1>
     <!-- Neck -->
-    <xacro:sara_neck_v1 name="neck" parent="torso_link">
-    	<origin xyz="0 0 0"
-    		    rpy="1.5708 0 1.5708"/>
+    <xacro:sara_neck_v1 name="neck" parent="torso">
+        <origin xyz="0 0 0"
+                rpy="1.5708 0 1.5708"/>
     </xacro:sara_neck_v1>
     <!-- Head -->
-    <xacro:sara_head_v1 name="head" parent="neck_link">
+    <xacro:sara_head_v1 name="head" parent="neck">
         <origin xyz="0.0 0.0 0.0"
-        	    rpy="1.5708 -1.5708 1.5708"/>
+                rpy="1.5708 -1.5708 1.5708"/>
     </xacro:sara_head_v1>
+    <!-- Shoulder -->
+    <xacro:sara_shoulder_v1 name="shoulder" parent="torso">
+        <origin xyz="0 0 0" rpy="0 3.1416 0"/>
+    </xacro:sara_shoulder_v1>
+    <!-- Arm -->
+    <xacro:sara_arm_v1 name="arm" parent="shoulder">
+        <origin xyz="0 0 0" rpy="1.5708 -1.5708 1.5708" />
+    </xacro:sara_arm_v1>
 </robot>

File: sara_description/urdf/sara_old.urdf.xacro (robot description, xacro)
@@ -258,5 +258,5 @@
 				<sphere radius="0.01" />
 			</geometry>
-			<origin xyz="0 0 0" rpy="0 0 0" />
+			<origin xyz="0 0.05 0" rpy="0 0 0" />
 		</visual>
 	</link>
