Commit message: Sara fonctionnelle dans gazebo. Sauf la pince qui a besoin d'amour

File: sara_description/urdf/arm_v1/arm.gazebo.xacro (robot description, xacro)
@@ -1,14 +1,23 @@
 <?xml version="1.0"?>
 <robot xmlns:xacro="http://ros.org/wiki/xacro">
-   <xacro:macro name="sara_arm_gazebo_v1">
-      <gazebo reference="arm_raise_link">
+   <xacro:macro name="sara_arm_gazebo_v1" params="name parent">
+       <gazebo reference="${name}_clavicular_link">
          <gravity>false</gravity>
-      </gazebo>
-      <gazebo reference="arm_rot_link">
+       </gazebo>
+       <gazebo reference="$${name}_fix_upper_link">
          <gravity>false</gravity>
-      </gazebo>
-      <gazebo reference="grasp_link">
+       </gazebo>
+       <gazebo reference="${name}_rot_upper_link">
          <gravity>false</gravity>
-      </gazebo>
-   </xacro:macro>
+       </gazebo>
+       <gazebo reference="${name}_fix_lower_link">
+         <gravity>false</gravity>
+       </gazebo>
+       <gazebo reference="${name}_rot_lower_link">
+         <gravity>false</gravity>
+       </gazebo>
+       <gazebo reference="grasp_link">
+         <gravity>false</gravity>
+       </gazebo>
+  </xacro:macro>
 </robot>

File: sara_description/urdf/arm_v1/arm.urdf.xacro (robot description, xacro)
@@ -1,9 +1,90 @@
 <?xml version="1.0"?>
 <robot xmlns:xacro="http://ros.org/wiki/xacro" >
-   <xacro:include filename="$(find sara_description)/urdf/robotiq_c2_model_macro.xacro" />
    <xacro:include filename="$(find sara_description)/urdf/arm_v1/arm.gazebo.xacro" />
-   <xacro:macro name="sara_arm_v1" params="name parent">
-      <!-- Link and joint to raise arm at elbow level -->
-      <link name="${name}_raise_link">
+   <xacro:macro name="sara_arm_v1" params="name parent end_effector">
+       <xacro:sara_arm_gazebo_v1 name="${name}" parent="${parent}"/>
+       <!-- Link and joint to raise arm at shoulder level -->
+      <link name="${name}_clavicular_link">
+         <visual>
+            <geometry>
+               <mesh filename="package://sara_description/meshes/epaule.dae" scale="0.001 0.001 0.001"/>
+            </geometry>
+            <origin xyz="0 0 0" rpy="0 3.1416 0"/>
+         </visual>
+         <collision>
+            <geometry>
+               <mesh filename="package://sara_description/meshes/epaule.dae" scale="0.001 0.001 0.001"/>
+            </geometry>
+            <origin xyz="0 0 0" rpy="0 3.1416 0"/>
+        </collision>
+        <inertial>
+            <mass value="1" />
+            <origin xyz="0 0 0" rpy="0 3.1416 0" />
+            <inertia ixx="0.001" ixy="0" ixz="0" iyy="0.001" iyz="0" izz="0.001" />
+        </inertial>
+      </link>
+      <joint name="${parent}_${name}_joint" type="revolute">
+         <parent link="${parent}_link"/>
+         <child link="${name}_clavicular_link"/>
+         <limit effort="1000.0" lower="-0.18" upper="1.21" velocity="0.5"/>
+         <origin xyz="0.008948 -0.145 0.155" rpy="0 -1.57 0" />
+         <axis xyz="0 0 1" />
+      </joint>
+      <!-- Link and joint to rotate the upper part of the arm at shoulder level -->
+      <link name="${name}_fix_upper_link">
+         <visual>
+            <geometry>
+               <mesh filename="package://sara_description/meshes/epaule.dae" scale="0.001 0.001 0.001"/>
+            </geometry>
+            <origin xyz="0 0 0" rpy="3.1416 0 1.5708"/>
+         </visual>
+         <collision>
+            <geometry>
+               <mesh filename="package://sara_description/meshes/epaule.dae" scale="0.001 0.001 0.001"/>
+            </geometry>
+            <origin xyz="0 0 0" rpy="3.1416 0 1.5708"/>
+         </collision>
+         <inertial>
+            <mass value="1" />
+            <origin xyz="0 0 0" rpy="3.1416 0 1.5708" />
+            <inertia ixx="0.001" ixy="0" ixz="0" iyy="0.001" iyz="0" izz="0.001" />
+        </inertial>
+      </link>
+      <joint name="${name}_shoulder_joint" type="revolute">
+         <parent link="${name}_clavicular_link"/>
+         <child link="${name}_fix_upper_link"/>
+         <limit effort="1000.0" lower="-3.29" upper="0.37" velocity="0.5"/>
+         <origin xyz="0 -0.085 0" rpy="-1.57 0 0" />
+         <axis xyz="0 0 1" />
+      </joint>
+      <!-- Link and joint to rotate the lower part of the arm at shoulder level -->
+      <link name="${name}_rot_upper_link">
+         <visual>
+            <geometry>
+               <mesh filename="package://sara_description/meshes/bras_haut.dae" scale="0.001 0.001 0.001"/>
+            </geometry>
+            <origin xyz="0 0 0" rpy="1.5708 3.1416 3.1416"/>
+         </visual>
+         <collision>
+            <geometry>
+               <mesh filename="package://sara_description/meshes/bras_haut.dae" scale="0.001 0.001 0.001"/>
+            </geometry>
+            <origin xyz="0 0 0" rpy="1.5708 3.1416 3.1416"/>
+         </collision>
+        <inertial>
+            <mass value="1" />
+            <origin xyz="0 0 0" rpy="1.5708 3.1416 3.1416" />
+            <inertia ixx="0.001" ixy="0" ixz="0" iyy="0.001" iyz="0" izz="0.001" />
+        </inertial>
+      </link>
+      <joint name="${name}_rot_elbow_joint" type="revolute">
+         <parent link="${name}_fix_upper_link"/>
+         <child link="${name}_rot_upper_link"/>
+         <limit effort="1000.0" lower="-2.14" upper="1.00" velocity="0.5"/>
+         <origin xyz="-0.085 0 0" rpy="1.5708 0 1.5708" />
+         <axis xyz="0 0 1" />
+      </joint>
+       <!-- Link and joint to raise arm at elbow level -->
+      <link name="${name}_fix_lower_link">
          <visual>
             <geometry>
@@ -18,8 +99,13 @@
             <origin xyz="0 0 -0.0005" rpy="3.1416 0 0"/>
          </collision>
-      </link>
-      <joint name="${name}_raise_joint" type="revolute">
-         <parent link="${parent}_lower_link"/>
-         <child link="${name}_raise_link"/>
+         <inertial>
+            <mass value="1" />
+            <origin xyz="0 0 0" rpy="0 3.1416 0" />
+            <inertia ixx="0.001" ixy="0" ixz="0" iyy="0.001" iyz="0" izz="0.001" />
+        </inertial>
+     </link>
+      <joint name="${name}_elbow_joint" type="revolute">
+         <parent link="${name}_rot_upper_link"/>
+         <child link="${name}_fix_lower_link"/>
          <limit effort="1000.0" lower="-2.20" upper="1.90" velocity="0.5"/>
          <origin xyz="0 0 -0.31" rpy="-1.5708 0 0" />
@@ -27,5 +113,5 @@
       </joint>
       <!-- Link and joint to rotate arm at elbow level -->
-      <link name="${name}_rot_link">
+      <link name="${name}_rot_lower_link">
          <visual>
             <geometry>
@@ -40,22 +126,23 @@
             <origin xyz="0 0 0" rpy="-1.5708 0 -1.5708"/>
          </collision>
-      </link>
-      <joint name="${name}_rot_joint" type="revolute">
-         <parent link="${name}_raise_link"/>
-         <child link="${name}_rot_link"/>
+          <inertial>
+            <mass value="1" />
+            <origin xyz="0 0 0" rpy="-1.5708 0 -1.5708" />
+            <inertia ixx="0.001" ixy="0" ixz="0" iyy="0.001" iyz="0" izz="0.001" />
+        </inertial>
+     </link>
+      <joint name="${name}_rot_wrist_joint" type="revolute">
+         <parent link="${name}_fix_lower_link"/>
+         <child link="${name}_rot_lower_link"/>
          <limit effort="1000.0" lower="-3.1416" upper="3.1416" velocity="0.5"/>
          <origin xyz="0 0.0945 0" rpy="1.5708 -1.5708 0" />
          <axis xyz="0 0 1" />
-      </joint>
-      <!-- Link and joint for wrist -->
-      <xacro:robotiq_c2_model prefix="">
-         <origin xyz="0 0 0" rpy="0 0 0" />
-      </xacro:robotiq_c2_model>
-      <joint name="${name}_wrist_joint" type="revolute">
-         <parent link="${name}_rot_link"/>
-         <child link="robotiq_85_base_link"/>
+     </joint>
+      <joint name="${name}_end_effector_joint" type="fixed">
+         <parent link="${name}_rot_lower_link"/>
+         <child link="${end_effector}_link"/>
          <limit effort="1000.0" lower="-0.26" upper="0.26" velocity="0.5" />
          <axis xyz="0 1 0"/>
-         <origin xyz="0 0 -0.10624" rpy="0 1.5708 1.5708"/>
+         <origin xyz="0 -0.004 -0.10624" rpy="0 1.5708 1.5708"/>
       </joint>
       <!-- Link and joint for target (grasp) -->
@@ -67,11 +154,15 @@
             <origin xyz="0 0.05 0" rpy="0 0 0" />
          </visual>
+         <inertial>
+            <mass value="0" />
+            <origin xyz="0 0 0" rpy="0 0 0" />
+            <inertia ixx="0.001" ixy="0" ixz="0" iyy="0.001" iyz="0" izz="0.001" />
+        </inertial>
       </link>
       <joint name="grasp_joint" type="fixed" >
-         <parent link="robotiq_85_base_link" />
+          <parent link="${end_effector}_link" />
          <child link="grasp_link" />
          <origin xyz="0.075 0 -0.012" rpy="3.1416 0 1.5708" />
       </joint>
-      <xacro:sara_arm_gazebo_v1 />
    </xacro:macro>
 </robot>

File: sara_description/urdf/base_v1/base.gazebo.xacro (robot description, xacro)
@@ -1,10 +1,10 @@
 <?xml version="1.0"?>
 <robot xmlns:xacro="http://ros.org/wiki/xacro">
-   <xacro:macro name="sara_base_gazebo_v1">
-      <gazebo reference="base_link">
+   <xacro:macro name="sara_base_gazebo_v1" params="name parent">
+       <gazebo reference="{name}_link">
          <gravity>false</gravity>
       </gazebo>
       <gazebo reference="spine_link">
-         <gravity>false</gravity>
+          <gravity>false</gravity>
       </gazebo>
       <!-- hokuyo -->

File: sara_description/urdf/base_v1/base.urdf.xacro (robot description, xacro)
@@ -1,30 +1,9 @@
 <?xml version="1.0"?>
 <robot xmlns:xacro="http://ros.org/wiki/xacro" >
+  <xacro:include filename="$(find sara_description)/urdf/base_v1/base.gazebo.xacro"/>
   <xacro:macro name="sara_base_v1" params="name parent">
-    <!-- Lien entre le torse et la colonne vertebrale -->
-    <link name="spine_link">
-      <visual>
-        <geometry>
-          <cylinder length="0.9" radius="0.04"/>
-        </geometry>
-        <origin xyz="0 0 0.49" rpy="0 0 0"/>
-        <material name="grey">
-          <color rgba="0.62 0.62 0.62 1"/>
-        </material>
-      </visual>
-      <collision>
-        <geometry>
-          <cylinder length="0.9" radius="0.07"/>
-        </geometry>
-        <origin xyz="0 0 0.49" rpy="0 0 0"/>
-      </collision>
-      <inertial>
-        <mass value="10"/>
-        <origin xyz="0 0 0.49" rpy="0 0 0"/>
-        <inertia ixx="0.001" ixy="0" ixz="0" iyy="0.001" iyz="0" izz="0.001"/>
-      </inertial>
-    </link>
-    <!-- Lien entre la colonne vertebrale et la base-->
-    <link name="base_link">
+    <xacro:sara_base_gazebo_v1 name="${name}" parent="${parent}"/>
+    <!-- Lien entre la base et la colonne vertebral-->
+    <link name="${name}_link">
       <visual>
         <geometry>
@@ -60,5 +39,5 @@
       </inertial>
     </link>
-    <joint name="base_spine_joint" type="fixed">
+    <joint name="${name}_spine_joint" type="fixed">
       <parent link="base_link"/>
       <child link="spine_link"/>
@@ -66,4 +45,27 @@
       <axis xyz="0 0 1" />
     </joint>
+  <!-- Lien entre le torse et la colonne vertebrale -->
+    <link name="spine_link">
+      <visual>
+        <geometry>
+          <cylinder length="0.9" radius="0.04"/>
+        </geometry>
+        <origin xyz="0 0 0.49" rpy="0 0 0"/>
+        <material name="grey">
+          <color rgba="0.62 0.62 0.62 1"/>
+        </material>
+      </visual>
+      <collision>
+        <geometry>
+          <cylinder length="0.9" radius="0.07"/>
+        </geometry>
+        <origin xyz="0 0 0.49" rpy="0 0 0"/>
+      </collision>
+      <inertial>
+        <mass value="10"/>
+        <origin xyz="0 0 0.49" rpy="0 0 0"/>
+        <inertia ixx="0.001" ixy="0" ixz="0" iyy="0.001" iyz="0" izz="0.001"/>
+      </inertial>
+    </link>
     <!-- Lidar -->
     <link name="lidar_link">

File: sara_description/urdf/head_v1/head.gazebo.xacro (robot description, xacro)
@@ -1,5 +1,5 @@
 <?xml version="1.0"?>
 <robot xmlns:xacro="http://ros.org/wiki/xacro">
-   <xacro:macro name="sara_head_gazebo_v1">
+   <xacro:macro name="sara_head_gazebo_v1" params="name parent">
       <gazebo reference="neck_dynamixel_link">
          <gravity>false</gravity>

File: sara_description/urdf/head_v1/head.urdf.xacro (robot description, xacro)
@@ -3,5 +3,6 @@
    <xacro:include filename="$(find sara_description)/urdf/head_v1/head.gazebo.xacro" />
    <xacro:macro name="sara_head_v1" params="name parent">
-      <link name="${name}_link">
+     <xacro:sara_head_gazebo_v1 name="${name}" parent="${parent}"/>
+     <link name="${name}_link">
          <visual>
             <geometry>
@@ -31,5 +32,10 @@
                <color rgba="0 0 1 1"/>
             </material>
-         </visual>
+        </visual>
+        <inertial>
+            <mass value="5" />
+            <origin xyz="0 0 0.018" rpy="0 0 0" />
+            <inertia ixx="0.001" ixy="0" ixz="0" iyy="0.001" iyz="0" izz="0.001" />
+         </inertial>
       </link>
       <joint name="${name}_dynamixel_joint" type="revolute">
@@ -40,5 +46,5 @@
          <axis xyz="0 0 1"/>
       </joint>
-      <joint name="${name}_neck_joint" type="revolute">
+      <joint name="${parent}_${name}_joint" type="revolute">
          <parent link="${parent}_link"/>
          <child link="${name}_link"/>
@@ -68,5 +74,4 @@
          <axis xyz="0 1 0" />
       </joint>
-      <xacro:sara_head_gazebo_v1 />
    </xacro:macro>
 </robot>

File: sara_description/urdf/neck_v1/neck.gazebo.xacro (robot description, xacro)
@@ -1,6 +1,6 @@
 <?xml version="1.0"?>
 <robot xmlns:xacro="http://ros.org/wiki/xacro">
-   <xacro:macro name="sara_neck_gazebo_v1">
-      <gazebo reference="neck_link">
+   <xacro:macro name="sara_neck_gazebo_v1" params="name parent">
+      <gazebo reference="${name}_link">
          <gravity>false</gravity>
       </gazebo>

File: sara_description/urdf/neck_v1/neck.urdf.xacro (robot description, xacro)
@@ -3,5 +3,6 @@
    <xacro:include filename="$(find sara_description)/urdf/neck_v1/neck.gazebo.xacro" />
    <xacro:macro name="sara_neck_v1" params="name parent">
-      <link name="${name}_link">
+     <xacro:sara_neck_gazebo_v1 name="${name}" parent="${parent}"/>
+     <link name="${name}_link">
          <visual>
             <geometry>
@@ -24,5 +25,4 @@
          <axis xyz="0 0 1"/>
       </joint>
-      <xacro:sara_neck_gazebo_v1 />
    </xacro:macro>
 </robot>

File: sara_description/urdf/robotiq_c2_model/robotiq_c2_model.xacro (robot description, xacro)
@@ -5,5 +5,5 @@
  -->
 <robot name="robotiq_c2_model" xmlns:xacro="http://ros.org/wiki/xacro">
-    <xacro:include filename="$(find sara_description)/urdf/robotiq_c2_model_macro.xacro" />
+    <xacro:include filename="$(find sara_description)/urdf/robotiq_c2_model/robotiq_c2_model_macro.xacro" />
     <xacro:robotiq_c2_model prefix=""/>
 </robot>

File: sara_description/urdf/robotiq_c2_model/robotiq_c2_model_macro.xacro (robot description, xacro)
@@ -8,4 +8,5 @@
 <robot xmlns:xacro="http://ros.org/wiki/xacro">
   <xacro:macro name="robotiq_c2_model" params="prefix">
+  <xacro:robotic_c2_model_gazebo prefix="${prefix}"/>
   <link name="${prefix}robotiq_85_base_link">
     <visual>
@@ -21,4 +22,9 @@
       <origin rpy="1.5707 0 1.5707" xyz="0 0 0"/>
     </collision>
+    <inertial>
+      <mass value="0.1" />
+      <origin xyz="0 0 0" rpy="1.5708 0 1.5708" />
+      <inertia ixx="0.001" ixy="0" ixz="0" iyy="0.001" iyz="0" izz="0.001" />
+    </inertial>
   </link>
   <joint name="${prefix}robotiq_85_left_knuckle_joint" type="revolute">
@@ -50,4 +56,9 @@
       <origin rpy="1.5707 -1.5707 0" xyz="0 .04191 -.0306"/>
     </collision>
+    <inertial>
+      <mass value="0.1" />
+      <origin xyz="0 0 0" rpy="1.5708 -1.5708 0"/>
+      <inertia ixx="0.001" ixy="0" ixz="0" iyy="0.001" iyz="0" izz="0.001" />
+    </inertial>
   </link>
   <link name="${prefix}robotiq_85_right_knuckle_link">
@@ -64,4 +75,9 @@
       <origin rpy="1.5707 1.5707 0" xyz="0 .04191 -.0306"/>
     </collision>
+    <inertial>
+      <mass value="0.1" />
+      <origin xyz="0 0 0" rpy="1.5708 1.5708 0" />
+      <inertia ixx="0.001" ixy="0" ixz="0" iyy="0.001" iyz="0" izz="0.001" />
+    </inertial>
   </link>
   <joint name="${prefix}robotiq_85_left_finger_joint" type="fixed">
@@ -92,4 +108,9 @@
       <origin rpy="-1.5707 1.5707 0" xyz="0 -.03683 .06194"/>
     </collision>
+    <inertial>
+      <mass value="0.1" />
+      <origin xyz="0 0 0" rpy="-1.5708 1.5708 0" />
+      <inertia ixx="0.001" ixy="0" ixz="0" iyy="0.001" iyz="0" izz="0.001" />
+    </inertial>
   </link>
   <link name="${prefix}robotiq_85_right_finger_link">
@@ -106,4 +127,9 @@
       <origin rpy="-1.5707 -1.5707 0" xyz="0 -.03683 .06194"/>
     </collision>
+    <inertial>
+      <mass value="0.1" />
+      <origin xyz="0 0 0" rpy="-1.5707 -1.5707 0" />
+      <inertia ixx="0.001" ixy="0" ixz="0" iyy="0.001" iyz="0" izz="0.001" />
+    </inertial>
   </link>
   <joint name="${prefix}robotiq_85_left_inner_knuckle_joint" type="revolute">
@@ -136,4 +162,9 @@
       <origin rpy="-1.5707 1.5707 0" xyz="0 -.04843 .0127"/>
     </collision>
+    <inertial>
+      <mass value="0.1" />
+      <origin xyz="0 0 0" rpy="-1.5707 1.5707 0" />
+      <inertia ixx="0.001" ixy="0" ixz="0" iyy="0.001" iyz="0" izz="0.001" />
+    </inertial>
   </link>
   <link name="${prefix}robotiq_85_right_inner_knuckle_link">
@@ -150,4 +181,9 @@
       <origin rpy="-1.5707 -1.5707 0" xyz="0 -.04843 .0127"/>
     </collision>
+    <inertial>
+      <mass value="0.1" />
+      <origin xyz="0 0 0" rpy="-1.5707 -1.5707 0" />
+      <inertia ixx="0.001" ixy="0" ixz="0" iyy="0.001" iyz="0" izz="0.001" />
+    </inertial>
   </link>
   <joint name="${prefix}robotiq_85_left_finger_tip_joint" type="revolute">
@@ -180,4 +216,9 @@
       <origin rpy="-1.5707 1.5707 0" xyz="0 -.090381 .051505"/>
     </collision>
+    <inertial>
+      <mass value="0.1" />
+      <origin xyz="0 0 0" rpy="-1.5707 1.5707 0" />
+      <inertia ixx="0.001" ixy="0" ixz="0" iyy="0.001" iyz="0" izz="0.001" />
+    </inertial>
   </link>
   <link name="${prefix}robotiq_85_right_finger_tip_link">
@@ -194,4 +235,9 @@
       <origin rpy="-1.5707 -1.5707 0" xyz="0 -.090381 .051505"/>
     </collision>
+    <inertial>
+      <mass value="0.1" />
+      <origin xyz="0 0 0" rpy="-1.5707 -1.5707 0" />
+      <inertia ixx="0.001" ixy="0" ixz="0" iyy="0.001" iyz="0" izz="0.001" />
+    </inertial>
   </link>
   </xacro:macro>

File: sara_description/urdf/sara.urdf.xacro (robot description, xacro)
@@ -5,5 +5,5 @@
     <xacro:include filename="$(find sara_description)/urdf/neck_v1/neck.urdf.xacro"/>
     <xacro:include filename="$(find sara_description)/urdf/head_v1/head.urdf.xacro"/>
-    <xacro:include filename="$(find sara_description)/urdf/shoulder_v1/shoulder.urdf.xacro"/>
+    <xacro:include filename="$(find sara_description)/urdf/robotiq_c2_model/robotiq_c2_model_macro.xacro"/>
     <xacro:include filename="$(find sara_description)/urdf/arm_v1/arm.urdf.xacro"/>
     <xacro:include filename="$(find sara_description)/urdf/base_v1/base.urdf.xacro"/>
@@ -14,8 +14,8 @@
     <!-- Head -->
     <xacro:sara_head_v1 name="head" parent="neck"/>
-    <!-- Shoulder -->
-    <xacro:sara_shoulder_v1 name="shoulder" parent="torso"/>
     <!-- Arm -->
-    <xacro:sara_arm_v1 name="arm" parent="shoulder"/>
+    <xacro:sara_arm_v1 name="arm" parent="torso" end_effector="robotiq_85_base"/>
+    <!-- End Effector -->
+    <xacro:robotiq_c2_model prefix=""/>
     <!-- Base -->
     <xacro:sara_base_v1 name="base" parent=""/>

File: sara_description/urdf/torso_v1/torso.gazebo.xacro (robot description, xacro)
@@ -1,6 +1,6 @@
 <?xml version="1.0"?>
 <robot xmlns:xacro="http://ros.org/wiki/xacro">
-   <xacro:macro name="sara_torso_gazebo_v1">
-      <gazebo reference="torso_link">
+   <xacro:macro name="sara_torso_gazebo_v1" params="name parent">
+      <gazebo reference="${name}_link">
          <gravity>false</gravity>
       </gazebo>

File: sara_description/urdf/torso_v1/torso.urdf.xacro (robot description, xacro)
@@ -3,5 +3,6 @@
    <xacro:include filename="$(find sara_description)/urdf/torso_v1/torso.gazebo.xacro" />
    <xacro:macro name="sara_torso_v1" params="name parent">
-      <link name="${name}_link">
+       <xacro:sara_torso_gazebo_v1 name="${name}" parent="${parent}"/>
+       <link name="${name}_link">
          <visual>
             <geometry>
@@ -25,5 +26,5 @@
          </inertial>
      </link>
-     <joint name="spine_torso_joint" type="fixed">
+     <joint name="${parent}_${name}_joint" type="fixed">
          <parent link="${parent}_link"/>
          <child link="${name}_link"/>
