Commit message: Merged the arm into a single urdf file

File: sara_description/urdf/arm_v1/arm.gazebo.xacro (robot description, xacro)
@@ -2,4 +2,13 @@
 <robot xmlns:xacro="http://ros.org/wiki/xacro">
    <xacro:macro name="sara_arm_gazebo_v1">
+      <gazebo reference="shoulder_raise_link">
+         <gravity>false</gravity>
+      </gazebo>
+      <gazebo reference="shoulder_upper_link">
+         <gravity>false</gravity>
+      </gazebo>
+      <gazebo reference="shoulder_lower_link">
+         <gravity>false</gravity>
+      </gazebo>
       <gazebo reference="arm_raise_link">
          <gravity>false</gravity>

File: sara_description/urdf/arm_v1/arm.urdf.xacro (robot description, xacro)
@@ -4,6 +4,72 @@
    <xacro:include filename="$(find sara_description)/urdf/arm_v1/arm.gazebo.xacro" />
    <xacro:macro name="sara_arm_v1" params="name parent">
+      <!-- Link and joint to raise arm at shoulder level -->
+      <link name="shoulder_raise_link">
+         <visual>
+            <geometry>
+               <mesh filename="package://sara_description/meshes/epaule.dae" scale="0.001 0.001 0.001"/>
+            </geometry>
+            <origin xyz="0 0 0" rpy="0 3.1416 0"/>
+         </visual>
+         <collision>
+            <geometry>
+               <mesh filename="package://sara_description/meshes/epaule.dae" scale="0.001 0.001 0.001"/>
+            </geometry>
+            <origin xyz="0 0 0" rpy="0 3.1416 0"/>
+         </collision>
+      </link>
+      <joint name="shoulder_raise_joint" type="revolute">
+         <parent link="${parent}_link"/>
+         <child link="shoulder_raise_link"/>
+         <limit effort="1000.0" lower="-0.18" upper="1.21" velocity="0.5"/>
+         <origin xyz="0.008948 -0.145 0.155" rpy="0 -1.57 0" />
+         <axis xyz="0 0 1" />
+      </joint>
+      <!-- Link and joint to rotate the upper part of the arm at shoulder level -->
+      <link name="shoulder_upper_link">
+         <visual>
+            <geometry>
+               <mesh filename="package://sara_description/meshes/epaule.dae" scale="0.001 0.001 0.001"/>
+            </geometry>
+            <origin xyz="0 0 0" rpy="3.1416 0 1.5708"/>
+         </visual>
+         <collision>
+            <geometry>
+               <mesh filename="package://sara_description/meshes/epaule.dae" scale="0.001 0.001 0.001"/>
+            </geometry>
+            <origin xyz="0 0 0" rpy="3.1416 0 1.5708"/>
+         </collision>
+      </link>
+      <joint name="shoulder_upper_joint" type="revolute">
+         <parent link="shoulder_raise_link"/>
+         <child link="shoulder_upper_link"/>
+         <limit effort="1000.0" lower="-3.29" upper="0.37" velocity="0.5"/>
+         <origin xyz="0 -0.085 0" rpy="-1.57 0 0" />
+         <axis xyz="0 0 1" />
+      </joint>
+      <!-- Link and joint to rotate the lower part of the arm at shoulder level -->
+      <link name="shoulder_lower_link">
+         <visual>
+            <geometry>
+               <mesh filename="package://sara_description/meshes/bras_haut.dae" scale="0.001 0.001 0.001"/>
+            </geometry>
+            <origin xyz="0 0 0" rpy="1.5708 3.1416 3.1416"/>
+         </visual>
+         <collision>
+            <geometry>
+               <mesh filename="package://sara_description/meshes/bras_haut.dae" scale="0.001 0.001 0.001"/>
+            </geometry>
+            <origin xyz="0 0 0" rpy="1.5708 3.1416 3.1416"/>
+         </collision>
+      </link>
+      <joint name="shoulder_lower_joint" type="revolute">
+         <parent link="shoulder_upper_link"/>
+         <child link="shoulder_lower_link"/>
+         <limit effort="1000.0" lower="-2.14" upper="1.00" velocity="0.5"/>
+         <origin xyz="-0.085 0 0" rpy="1.5708 0 1.5708" />
+         <axis xyz="0 0 1" />
+      </joint>
       <!-- Link and joint to raise arm at elbow level -->
-      <link name="${name}_raise_link">
+      <link name="arm_raise_link">
          <visual>
             <geometry>
@@ -19,7 +85,7 @@
          </collision>
       </link>
-      <joint name="${name}_raise_joint" type="revolute">
-         <parent link="${parent}_lower_link"/>
-         <child link="${name}_raise_link"/>
+      <joint name="arm_raise_joint" type="revolute">
+         <parent link="shoulder_lower_link"/>
+         <child link="arm_raise_link"/>
          <limit effort="1000.0" lower="-2.20" upper="1.90" velocity="0.5"/>
          <origin xyz="0 0 -0.31" rpy="-1.5708 0 0" />
@@ -27,5 +93,5 @@
       </joint>
       <!-- Link and joint to rotate arm at elbow level -->
-      <link name="${name}_rot_link">
+      <link name="arm_rot_link">
          <visual>
             <geometry>
@@ -41,7 +107,7 @@
          </collision>
       </link>
-      <joint name="${name}_rot_joint" type="revolute">
-         <parent link="${name}_raise_link"/>
-         <child link="${name}_rot_link"/>
+      <joint name="arm_rot_joint" type="revolute">
+         <parent link="arm_raise_link"/>
+         <child link="arm_rot_link"/>
          <limit effort="1000.0" lower="-3.1416" upper="3.1416" velocity="0.5"/>
          <origin xyz="0 0.0945 0" rpy="1.5708 -1.5708 0" />
@@ -52,6 +118,6 @@
          <origin xyz="0 0 0" rpy="0 0 0" />
       </xacro:robotiq_c2_model>
-      <joint name="${name}_wrist_joint" type="revolute">
-         <parent link="${name}_rot_link"/>
+      <joint name="arm_wrist_joint" type="revolute">
+         <parent link="arm_rot_link"/>
          <child link="robotiq_85_base_link"/>
          <limit effort="1000.0" lower="-0.26" upper="0.26" velocity="0.5" />

File: sara_description/urdf/sara.urdf.xacro (robot description, xacro)
@@ -5,7 +5,8 @@
     <xacro:include filename="$(find sara_description)/urdf/neck_v1/neck.urdf.xacro"/>
     <xacro:include filename="$(find sara_description)/urdf/head_v1/head.urdf.xacro"/>
-    <xacro:include filename="$(find sara_description)/urdf/shoulder_v1/shoulder.urdf.xacro"/>
     <xacro:include filename="$(find sara_description)/urdf/arm_v1/arm.urdf.xacro"/>
     <xacro:include filename="$(find sara_description)/urdf/base_v1/base.urdf.xacro"/>
+    <!-- Base -->
+    <xacro:sara_base_v1 name="base" parent=""/>
     <!-- Torso -->
     <xacro:sara_torso_v1 name="torso" parent="spine"/>
@@ -14,9 +15,5 @@
     <!-- Head -->
     <xacro:sara_head_v1 name="head" parent="neck"/>
-    <!-- Shoulder -->
-    <xacro:sara_shoulder_v1 name="shoulder" parent="torso"/>
     <!-- Arm -->
-    <xacro:sara_arm_v1 name="arm" parent="shoulder"/>
-    <!-- Base -->
-    <xacro:sara_base_v1 name="base" parent=""/>
+    <xacro:sara_arm_v1 name="arm" parent="torso"/>
 </robot>
