Commit message: Finalisation du nouveau format d'URDF en xacro
-Ajout de la base
-Cleanup
-TODO: Ajouter les tags gazebo

File: sara_description/urdf/arm_v1/arm.urdf.xacro (robot description, xacro)
@@ -2,5 +2,5 @@
 <robot xmlns:xacro="http://ros.org/wiki/xacro" >
     <xacro:include filename="$(find sara_description)/urdf/robotiq_c2_model_macro.xacro" />
-    <xacro:macro name="sara_arm_v1" params="name parent *origin">
+    <xacro:macro name="sara_arm_v1" params="name parent">
         <!-- Link and joint to raise arm at elbow level -->
         <link name="${name}_raise_link">

File: sara_description/urdf/head_v1/head.urdf.xacro (robot description, xacro)
@@ -1,5 +1,5 @@
 <?xml version="1.0"?>
 <robot xmlns:xacro="http://ros.org/wiki/xacro" >
-   <xacro:macro name="sara_head_v1" params="name parent *origin">
+   <xacro:macro name="sara_head_v1" params="name parent">
       <link name="${name}_link">
          <visual>
@@ -21,5 +21,5 @@
          </inertial>
       </link>
-      <link name="neck_dynamixel_link">
+      <link name="${parent}_dynamixel_link">
          <visual>
             <geometry>
@@ -33,5 +33,5 @@
       </link>
       <joint name="${name}_dynamixel_joint" type="revolute">
-         <parent link="neck_dynamixel_link"/>
+         <parent link="${parent}_dynamixel_link"/>
          <child link="${name}_link"/>
          <limit effort="1000.0" lower="-1.00" upper="0.40" velocity="0.5"/>
@@ -44,4 +44,25 @@
          <origin xyz="0 0 0.0927" rpy="1.57 0 0"/>
       </joint>
+      <!-- xtion -->
+      <link name="camera_link">
+         <visual>
+            <geometry>
+               <mesh filename="package://sara_description/meshes/xtion.dae" scale="0.001 0.001 0.001"/>
+            </geometry>
+            <origin xyz="0 0 0" rpy="1.5708 0 1.5708"/>
+            <material name="black"/>
+         </visual>
+         <inertial>
+            <mass value="0.5"/>
+            <origin xyz="0 0 0" rpy="1.5708 0 1.5708"/>
+            <inertia ixx="0.001" ixy="0" ixz="0" iyy="0.001" iyz="0" izz="0.001"/>
+         </inertial>
+      </link>
+      <joint name="camera_joint" type="fixed">
+         <parent link="${name}_link"/>
+         <child link="camera_link"/>
+         <origin xyz="0.0776104 -0.13 0" rpy="1.57 0 0" />
+         <axis xyz="0 1 0" />
+      </joint>
    </xacro:macro>
 </robot>

File: sara_description/urdf/neck_v1/neck.urdf.xacro (robot description, xacro)
@@ -1,5 +1,5 @@
 <?xml version="1.0"?>
 <robot xmlns:xacro="http://ros.org/wiki/xacro" >
-    <xacro:macro name="sara_neck_v1" params="name parent *origin">
+    <xacro:macro name="sara_neck_v1" params="name parent">
         <link name="${name}_link">
             <visual>

File: sara_description/urdf/sara.urdf.xacro (robot description, xacro)
@@ -2,31 +2,21 @@
 <robot xmlns:xacro="http://playerstage.sourceforge.net/gazebo/xmlschema/#interface" name="sara" >
     <!-- Inclure tous les autres urdf.xacros ici -->
-    <xacro:include filename="$(find sara_description)/urdf/torso_v1/torso.urdf.xacro" />
-    <xacro:include filename="$(find sara_description)/urdf/neck_v1/neck.urdf.xacro" />
-    <xacro:include filename="$(find sara_description)/urdf/head_v1/head.urdf.xacro" />
-    <xacro:include filename="$(find sara_description)/urdf/shoulder_v1/shoulder.urdf.xacro" />
-    <xacro:include filename="$(find sara_description)/urdf/arm_v1/arm.urdf.xacro" />
+    <xacro:include filename="$(find sara_description)/urdf/torso_v1/torso.urdf.xacro"/>
+    <xacro:include filename="$(find sara_description)/urdf/neck_v1/neck.urdf.xacro"/>
+    <xacro:include filename="$(find sara_description)/urdf/head_v1/head.urdf.xacro"/>
+    <xacro:include filename="$(find sara_description)/urdf/shoulder_v1/shoulder.urdf.xacro"/>
+    <xacro:include filename="$(find sara_description)/urdf/arm_v1/arm.urdf.xacro"/>
+    <xacro:include filename="$(find sara_description)/urdf/base_v1/base.urdf.xacro"/>
     <!-- Torso -->
-    <xacro:sara_torso_v1 name="torso" parent="">
-        <origin xyz="0 0 0"
-                rpy="1.5708 0 1.5708"/>
-    </xacro:sara_torso_v1>
+    <xacro:sara_torso_v1 name="torso" parent=""/>
     <!-- Neck -->
-    <xacro:sara_neck_v1 name="neck" parent="torso">
-        <origin xyz="0 0 0"
-                rpy="1.5708 0 1.5708"/>
-    </xacro:sara_neck_v1>
+    <xacro:sara_neck_v1 name="neck" parent="torso"/>
     <!-- Head -->
-    <xacro:sara_head_v1 name="head" parent="neck">
-        <origin xyz="0.0 0.0 0.0"
-                rpy="1.5708 -1.5708 1.5708"/>
-    </xacro:sara_head_v1>
+    <xacro:sara_head_v1 name="head" parent="neck"/>
     <!-- Shoulder -->
-    <xacro:sara_shoulder_v1 name="shoulder" parent="torso">
-        <origin xyz="0 0 0" rpy="0 3.1416 0"/>
-    </xacro:sara_shoulder_v1>
+    <xacro:sara_shoulder_v1 name="shoulder" parent="torso"/>
     <!-- Arm -->
-    <xacro:sara_arm_v1 name="arm" parent="shoulder">
-        <origin xyz="0 0 0" rpy="1.5708 -1.5708 1.5708" />
-    </xacro:sara_arm_v1>
+    <xacro:sara_arm_v1 name="arm" parent="shoulder"/>
+    <!-- Base -->
+    <xacro:sara_base_v1 name="base" parent="torso"/>
 </robot>

File: sara_description/urdf/shoulder_v1/shoulder.urdf.xacro (robot description, xacro)
@@ -1,5 +1,5 @@
 <?xml version="1.0"?>
 <robot xmlns:xacro="http://ros.org/wiki/xacro" >
-    <xacro:macro name="sara_shoulder_v1" params="name parent *origin">
+    <xacro:macro name="sara_shoulder_v1" params="name parent">
         <!-- Link and joint to raise arm at shoulder level -->
         <link name="${name}_raise_link">

File: sara_description/urdf/torso_v1/torso.urdf.xacro (robot description, xacro)
@@ -1,5 +1,5 @@
 <?xml version="1.0"?>
 <robot xmlns:xacro="http://ros.org/wiki/xacro" >
-   <xacro:macro name="sara_torso_v1" params="name parent *origin">
+   <xacro:macro name="sara_torso_v1" params="name parent">
       <link name="${name}_link">
          <visual>

Commit message: Ajout de gazebo
-Liens entre les fichiers: sara.urdf.xacro -> piece.urdf.xacro -> piece.gazebo.xacro

File: sara_description/urdf/arm_v1/arm.urdf.xacro (robot description, xacro)
@@ -1,75 +1,77 @@
 <?xml version="1.0"?>
 <robot xmlns:xacro="http://ros.org/wiki/xacro" >
-    <xacro:include filename="$(find sara_description)/urdf/robotiq_c2_model_macro.xacro" />
-    <xacro:macro name="sara_arm_v1" params="name parent">
-        <!-- Link and joint to raise arm at elbow level -->
-        <link name="${name}_raise_link">
-            <visual>
-                <geometry>
-                    <mesh filename="package://sara_description/meshes/coude.dae" scale="0.001 0.001 0.001"/>
-                </geometry>
-                <origin xyz="0 0 -0.0005" rpy="3.1416 0 0"/>
-            </visual>
-            <collision>
-                <geometry>
-                    <mesh filename="package://sara_description/meshes/coude.dae" scale="0.001 0.001 0.001"/>
-                </geometry>
-                <origin xyz="0 0 -0.0005" rpy="3.1416 0 0"/>
-            </collision>
-        </link>
-        <joint name="${name}_raise_joint" type="revolute">
-            <parent link="${parent}_lower_link"/>
-            <child link="${name}_raise_link"/>
-            <limit effort="1000.0" lower="-2.20" upper="1.90" velocity="0.5"/>
-            <origin xyz="0 0 -0.31" rpy="-1.5708 0 0" />
-            <axis xyz="0 0 1" />
-        </joint>
-        <!-- Link and joint to rotate arm at elbow level -->
-        <link name="${name}_rot_link">
-            <visual>
-                <geometry>
-                    <mesh filename="package://sara_description/meshes/avant-bras.dae" scale="0.001 0.001 0.001"/>
-                </geometry>
-                <origin xyz="0 0 0" rpy="-1.5708 0 -1.5708"/>
-            </visual>
-            <collision>
-                <geometry>
-                    <mesh filename="package://sara_description/meshes/avant-bras.dae" scale="0.001 0.001 0.001"/>
-                </geometry>
-                <origin xyz="0 0 0" rpy="-1.5708 0 -1.5708"/>
-            </collision>
-        </link>
-        <joint name="${name}_rot_joint" type="revolute">
-            <parent link="${name}_raise_link"/>
-            <child link="${name}_rot_link"/>
-            <limit effort="1000.0" lower="-3.1416" upper="3.1416" velocity="0.5"/>
-            <origin xyz="0 0.0945 0" rpy="1.5708 -1.5708 0" />
-            <axis xyz="0 0 1" />
-        </joint>
-        <!-- Link and joint for wrist -->
-        <xacro:robotiq_c2_model prefix="">
-            <origin xyz="0 0 0" rpy="0 0 0" />
-        </xacro:robotiq_c2_model>
-        <joint name="${name}_wrist_joint" type="revolute">
-            <parent link="${name}_rot_link"/>
-            <child link="robotiq_85_base_link"/>
-            <limit effort="1000.0" lower="-0.26" upper="0.26" velocity="0.5" />
-            <axis xyz="0 1 0"/>
-            <origin xyz="0 0 -0.10624" rpy="0 1.5708 1.5708"/>
-        </joint>
-        <!-- Link and joint for target (grasp) -->
-        <link name="grasp_link" >
-            <visual>
-                <geometry>
-                    <sphere radius="0.01" />
-                </geometry>
-                <origin xyz="0 0.05 0" rpy="0 0 0" />
-            </visual>
-        </link>
-        <joint name="grasp_joint" type="fixed" >
-            <parent link="robotiq_85_base_link" />
-            <child link="grasp_link" />
-            <origin xyz="0.075 0 -0.012" rpy="3.1416 0 1.5708" />
-        </joint>
-    </xacro:macro>
+   <xacro:include filename="$(find sara_description)/urdf/robotiq_c2_model_macro.xacro" />
+   <xacro:include filename="$(find sara_description)/urdf/arm_v1/arm.gazebo.xacro" />
+   <xacro:macro name="sara_arm_v1" params="name parent">
+      <!-- Link and joint to raise arm at elbow level -->
+      <link name="${name}_raise_link">
+         <visual>
+            <geometry>
+               <mesh filename="package://sara_description/meshes/coude.dae" scale="0.001 0.001 0.001"/>
+            </geometry>
+            <origin xyz="0 0 -0.0005" rpy="3.1416 0 0"/>
+         </visual>
+         <collision>
+            <geometry>
+               <mesh filename="package://sara_description/meshes/coude.dae" scale="0.001 0.001 0.001"/>
+            </geometry>
+            <origin xyz="0 0 -0.0005" rpy="3.1416 0 0"/>
+         </collision>
+      </link>
+      <joint name="${name}_raise_joint" type="revolute">
+         <parent link="${parent}_lower_link"/>
+         <child link="${name}_raise_link"/>
+         <limit effort="1000.0" lower="-2.20" upper="1.90" velocity="0.5"/>
+         <origin xyz="0 0 -0.31" rpy="-1.5708 0 0" />
+         <axis xyz="0 0 1" />
+      </joint>
+      <!-- Link and joint to rotate arm at elbow level -->
+      <link name="${name}_rot_link">
+         <visual>
+            <geometry>
+               <mesh filename="package://sara_description/meshes/avant-bras.dae" scale="0.001 0.001 0.001"/>
+            </geometry>
+            <origin xyz="0 0 0" rpy="-1.5708 0 -1.5708"/>
+         </visual>
+         <collision>
+            <geometry>
+               <mesh filename="package://sara_description/meshes/avant-bras.dae" scale="0.001 0.001 0.001"/>
+            </geometry>
+            <origin xyz="0 0 0" rpy="-1.5708 0 -1.5708"/>
+         </collision>
+      </link>
+      <joint name="${name}_rot_joint" type="revolute">
+         <parent link="${name}_raise_link"/>
+         <child link="${name}_rot_link"/>
+         <limit effort="1000.0" lower="-3.1416" upper="3.1416" velocity="0.5"/>
+         <origin xyz="0 0.0945 0" rpy="1.5708 -1.5708 0" />
+         <axis xyz="0 0 1" />
+      </joint>
+      <!-- Link and joint for wrist -->
+      <xacro:robotiq_c2_model prefix="">
+         <origin xyz="0 0 0" rpy="0 0 0" />
+      </xacro:robotiq_c2_model>
+      <joint name="${name}_wrist_joint" type="revolute">
+         <parent link="${name}_rot_link"/>
+         <child link="robotiq_85_base_link"/>
+         <limit effort="1000.0" lower="-0.26" upper="0.26" velocity="0.5" />
+         <axis xyz="0 1 0"/>
+         <origin xyz="0 0 -0.10624" rpy="0 1.5708 1.5708"/>
+      </joint>
+      <!-- Link and joint for target (grasp) -->
+      <link name="grasp_link" >
+         <visual>
+            <geometry>
+               <sphere radius="0.01" />
+            </geometry>
+            <origin xyz="0 0.05 0" rpy="0 0 0" />
+         </visual>
+      </link>
+      <joint name="grasp_joint" type="fixed" >
+         <parent link="robotiq_85_base_link" />
+         <child link="grasp_link" />
+         <origin xyz="0.075 0 -0.012" rpy="3.1416 0 1.5708" />
+      </joint>
+      <xacro:sara_arm_gazebo_v1 />
+   </xacro:macro>
 </robot>

File: sara_description/urdf/base_v1/base.urdf.xacro (robot description, xacro)
@@ -1,104 +1,106 @@
 <?xml version="1.0"?>
 <robot xmlns:xacro="http://ros.org/wiki/xacro" >
-  <xacro:macro name="sara_base_v1" params="name parent">
-    <!-- Lien entre le torse et la colonne vertebrale -->
-    <link name="spine_link">
-      <visual>
-        <geometry>
-          <cylinder length="0.9" radius="0.04"/>
-        </geometry>
-        <origin xyz="0 0 0.49" rpy="0 0 0"/>
-        <material name="grey">
-          <color rgba="0.62 0.62 0.62 1"/>
-        </material>
-      </visual>
-      <collision>
-        <geometry>
-          <cylinder length="0.9" radius="0.07"/>
-        </geometry>
-        <origin xyz="0 0 0.49" rpy="0 0 0"/>
-      </collision>
-      <inertial>
-        <mass value="10"/>
-        <origin xyz="0 0 0.49" rpy="0 0 0"/>
-        <inertia ixx="0.001" ixy="0" ixz="0" iyy="0.001" iyz="0" izz="0.001"/>
-      </inertial>
-    </link>
-    <joint name="spine_torso_joint" type="fixed">
-      <parent link="spine_link"/>
-      <child link="${parent}_link"/>
-      <limit effort="1000.0" lower="0" upper="0.5" velocity="0.2"/>
-      <origin xyz="0 0 1.112" rpy="0 0 0" />
-      <axis xyz="0 0 1" />
-    </joint>
-    <!-- Lien entre la colonne vertebrale et la base-->
-    <link name="base_link">
-      <visual>
-        <geometry>
-          <box size="0.7637 0.64311 0.14"/>
-        </geometry>
-        <origin xyz="0.0 0 0.07" rpy="0 0 0"/>
-        <material name="grey">
-          <color rgba="0.62 0.62 0.62 1"/>
-        </material>
-      </visual>
-      <visual>
-        <geometry>
-          <box size="0.55 0.64311 0.57"/>
-        </geometry>
-        <origin xyz="-0.115 0 0.42" rpy="0 0 0"/>
-      </visual>
-      <collision>
-        <geometry>
-          <box size="0.7637 0.64311 0.14"/>
-        </geometry>
-        <origin xyz="0.0 0 0.07" rpy="0 0 0"/>
-      </collision>
-      <collision>
-        <geometry>
-          <box size="0.55 0.64311 0.57"/>
-        </geometry>
-        <origin xyz="-0.115 0 0.42" rpy="0 0 0"/>
-      </collision>
-      <inertial>
-        <mass value="10"/>
-        <origin xyz="-0.115 0 0.42" rpy="0 0 0"/>
-        <inertia ixx="0.001" ixy="0" ixz="0" iyy="0.001" iyz="0" izz="0.001"/>
-      </inertial>
-    </link>
-    <joint name="base_spine_joint" type="fixed">
-      <parent link="base_link"/>
-      <child link="spine_link"/>
-      <origin xyz="0.2 0 0" rpy="0 0 0" />
-      <axis xyz="0 0 1" />
-    </joint>
-    <!-- Lidar -->
-    <link name="lidar_link">
-      <visual>
-        <geometry>
-          <cylinder length="0.1" radius="0.03"/>
-        </geometry>
-        <origin xyz="0 0 0" rpy="0 0 0"/>
-        <material name="orange">
-          <color rgba="1 0.5 0 1"/>
-        </material>
-      </visual>
-      <collision>
-        <geometry>
-          <cylinder length="0.1" radius="0.03"/>
-        </geometry>
-        <origin xyz="0 0 0" rpy="0 0 0"/>
-      </collision>
-      <inertial>
-        <mass value="0.5"/>
-        <origin xyz="0 0 0" rpy="0 0 0"/>
-        <inertia ixx="0.001" ixy="0" ixz="0" iyy="0.001" iyz="0" izz="0.001"/>
-      </inertial>
-    </link>
-    <joint name="laser_joint" type="fixed">
-      <parent link="base_link"/>
-      <child link="lidar_link"/>
-      <origin xyz="0.34 0 0.19" rpy="0 0 0" />
-    </joint>
-  </xacro:macro>
+   <xacro:include filename="$(find sara_description)/urdf/base_v1/base.gazebo.xacro" />
+   <xacro:macro name="sara_base_v1" params="name parent">
+      <!-- Lien entre le torse et la colonne vertebrale -->
+      <link name="spine_link">
+         <visual>
+            <geometry>
+               <cylinder length="0.9" radius="0.04"/>
+            </geometry>
+            <origin xyz="0 0 0.49" rpy="0 0 0"/>
+            <material name="grey">
+               <color rgba="0.62 0.62 0.62 1"/>
+            </material>
+         </visual>
+         <collision>
+            <geometry>
+               <cylinder length="0.9" radius="0.07"/>
+            </geometry>
+            <origin xyz="0 0 0.49" rpy="0 0 0"/>
+         </collision>
+         <inertial>
+            <mass value="10"/>
+            <origin xyz="0 0 0.49" rpy="0 0 0"/>
+            <inertia ixx="0.001" ixy="0" ixz="0" iyy="0.001" iyz="0" izz="0.001"/>
+         </inertial>
+      </link>
+      <joint name="spine_torso_joint" type="fixed">
+         <parent link="spine_link"/>
+         <child link="${parent}_link"/>
+         <limit effort="1000.0" lower="0" upper="0.5" velocity="0.2"/>
+         <origin xyz="0 0 1.112" rpy="0 0 0" />
+         <axis xyz="0 0 1" />
+      </joint>
+      <!-- Lien entre la colonne vertebrale et la base-->
+      <link name="base_link">
+         <visual>
+            <geometry>
+               <box size="0.7637 0.64311 0.14"/>
+            </geometry>
+            <origin xyz="0.0 0 0.07" rpy="0 0 0"/>
+            <material name="grey">
+               <color rgba="0.62 0.62 0.62 1"/>
+            </material>
+         </visual>
+         <visual>
+            <geometry>
+               <box size="0.55 0.64311 0.57"/>
+            </geometry>
+            <origin xyz="-0.115 0 0.42" rpy="0 0 0"/>
+         </visual>
+         <collision>
+            <geometry>
+               <box size="0.7637 0.64311 0.14"/>
+            </geometry>
+            <origin xyz="0.0 0 0.07" rpy="0 0 0"/>
+         </collision>
+         <collision>
+            <geometry>
+               <box size="0.55 0.64311 0.57"/>
+            </geometry>
+            <origin xyz="-0.115 0 0.42" rpy="0 0 0"/>
+         </collision>
+         <inertial>
+            <mass value="10"/>
+            <origin xyz="-0.115 0 0.42" rpy="0 0 0"/>
+            <inertia ixx="0.001" ixy="0" ixz="0" iyy="0.001" iyz="0" izz="0.001"/>
+         </inertial>
+      </link>
+      <joint name="base_spine_joint" type="fixed">
+         <parent link="base_link"/>
+         <child link="spine_link"/>
+         <origin xyz="0.2 0 0" rpy="0 0 0" />
+         <axis xyz="0 0 1" />
+      </joint>
+      <!-- Lidar -->
+      <link name="lidar_link">
+         <visual>
+            <geometry>
+               <cylinder length="0.1" radius="0.03"/>
+            </geometry>
+            <origin xyz="0 0 0" rpy="0 0 0"/>
+            <material name="orange">
+               <color rgba="1 0.5 0 1"/>
+            </material>
+         </visual>
+         <collision>
+            <geometry>
+               <cylinder length="0.1" radius="0.03"/>
+            </geometry>
+            <origin xyz="0 0 0" rpy="0 0 0"/>
+         </collision>
+         <inertial>
+            <mass value="0.5"/>
+            <origin xyz="0 0 0" rpy="0 0 0"/>
+            <inertia ixx="0.001" ixy="0" ixz="0" iyy="0.001" iyz="0" izz="0.001"/>
+         </inertial>
+      </link>
+      <joint name="laser_joint" type="fixed">
+         <parent link="base_link"/>
+         <child link="lidar_link"/>
+         <origin xyz="0.34 0 0.19" rpy="0 0 0" />
+      </joint>
+      <xacro:sara_base_gazebo_v1 />
+   </xacro:macro>
 </robot>

File: sara_description/urdf/head_v1/head.urdf.xacro (robot description, xacro)
@@ -1,4 +1,5 @@
 <?xml version="1.0"?>
 <robot xmlns:xacro="http://ros.org/wiki/xacro" >
+   <xacro:include filename="$(find sara_description)/urdf/head_v1/head.gazebo.xacro" />
    <xacro:macro name="sara_head_v1" params="name parent">
       <link name="${name}_link">
@@ -65,4 +66,5 @@
          <axis xyz="0 1 0" />
       </joint>
+      <xacro:sara_head_gazebo_v1 />
    </xacro:macro>
 </robot>

File: sara_description/urdf/neck_v1/neck.urdf.xacro (robot description, xacro)
@@ -1,26 +1,28 @@
 <?xml version="1.0"?>
 <robot xmlns:xacro="http://ros.org/wiki/xacro" >
-    <xacro:macro name="sara_neck_v1" params="name parent">
-        <link name="${name}_link">
-            <visual>
-                <geometry>
-                    <mesh filename="package://sara_description/meshes/cou.dae" scale="0.001 0.001 0.001"/>
-                </geometry>
-                <origin xyz="0 0 0" rpy="1.5708 0 1.5708"/>
-            </visual>
-            <inertial>
-                <mass value="2"/>
-                <origin xyz="0 0 0" rpy="1.5708 0 1.5708"/>
-                <inertia ixx="0.001" ixy="0" ixz="0" iyy="0.001" iyz="0" izz="0.001"/>
-            </inertial>
-        </link>
-        <joint name="${parent}_${name}_joint" type="revolute">
-            <parent link="${parent}_link"/>
-            <child link="${name}_link"/>
-            <limit effort="1000.0" lower="-1.22173" upper="1.22173" velocity="0.5"/>
-            <!-- 1mm ajoute en z (collision) -->
-            <origin xyz="0.032295 0 0.2438" rpy="0 0 0"/>
-            <axis xyz="0 0 1"/>
-        </joint>
-    </xacro:macro>
+   <xacro:include filename="$(find sara_description)/urdf/neck_v1/neck.gazebo.xacro" />
+   <xacro:macro name="sara_neck_v1" params="name parent">
+      <link name="${name}_link">
+         <visual>
+            <geometry>
+               <mesh filename="package://sara_description/meshes/cou.dae" scale="0.001 0.001 0.001"/>
+            </geometry>
+            <origin xyz="0 0 0" rpy="1.5708 0 1.5708"/>
+         </visual>
+         <inertial>
+            <mass value="2"/>
+            <origin xyz="0 0 0" rpy="1.5708 0 1.5708"/>
+            <inertia ixx="0.001" ixy="0" ixz="0" iyy="0.001" iyz="0" izz="0.001"/>
+         </inertial>
+      </link>
+      <joint name="${parent}_${name}_joint" type="revolute">
+         <parent link="${parent}_link"/>
+         <child link="${name}_link"/>
+         <limit effort="1000.0" lower="-1.22173" upper="1.22173" velocity="0.5"/>
+         <!-- 1mm ajoute en z (collision) -->
+         <origin xyz="0.032295 0 0.2438" rpy="0 0 0"/>
+         <axis xyz="0 0 1"/>
+      </joint>
+      <xacro:sara_neck_gazebo_v1 />
+   </xacro:macro>
 </robot>
