Commit message: Ajout de gazebo
-Liens entre les fichiers: sara.urdf.xacro -> piece.urdf.xacro -> piece.gazebo.xacro

File: sara_description/urdf/shoulder_v1/shoulder.urdf.xacro (robot description, xacro)
@@ -1,71 +1,73 @@
 <?xml version="1.0"?>
 <robot xmlns:xacro="http://ros.org/wiki/xacro" >
-    <xacro:macro name="sara_shoulder_v1" params="name parent">
-        <!-- Link and joint to raise arm at shoulder level -->
-        <link name="${name}_raise_link">
-            <visual>
-                <geometry>
-                    <mesh filename="package://sara_description/meshes/epaule.dae" scale="0.001 0.001 0.001"/>
-                </geometry>
-                <origin xyz="0 0 0" rpy="0 3.1416 0"/>
-            </visual>
-            <collision>
-                <geometry>
-                    <mesh filename="package://sara_description/meshes/epaule.dae" scale="0.001 0.001 0.001"/>
-                </geometry>
-                <origin xyz="0 0 0" rpy="0 3.1416 0"/>
-            </collision>
-        </link>
-        <joint name="${name}_raise_joint" type="revolute">
-            <parent link="${parent}_link"/>
-            <child link="${name}_raise_link"/>
-            <limit effort="1000.0" lower="-0.18" upper="1.21" velocity="0.5"/>
-            <origin xyz="0.008948 -0.145 0.155" rpy="0 -1.57 0" />
-            <axis xyz="0 0 1" />
-        </joint>
-        <!-- Link and joint to rotate the upper part of the arm at shoulder level -->
-        <link name="${name}_upper_link">
-            <visual>
-                <geometry>
-                    <mesh filename="package://sara_description/meshes/epaule.dae" scale="0.001 0.001 0.001"/>
-                </geometry>
-                <origin xyz="0 0 0" rpy="3.1416 0 1.5708"/>
-            </visual>
-            <collision>
-                <geometry>
-                    <mesh filename="package://sara_description/meshes/epaule.dae" scale="0.001 0.001 0.001"/>
-                </geometry>
-                <origin xyz="0 0 0" rpy="3.1416 0 1.5708"/>
-            </collision>
-        </link>
-        <joint name="${name}_upper_joint" type="revolute">
-            <parent link="${name}_raise_link"/>
-            <child link="${name}_upper_link"/>
-            <limit effort="1000.0" lower="-3.29" upper="0.37" velocity="0.5"/>
-            <origin xyz="0 -0.085 0" rpy="-1.57 0 0" />
-            <axis xyz="0 0 1" />
-        </joint>
-        <!-- Link and joint to rotate the lower part of the arm at shoulder level -->
-        <link name="${name}_lower_link">
-            <visual>
-                <geometry>
-                    <mesh filename="package://sara_description/meshes/bras_haut.dae" scale="0.001 0.001 0.001"/>
-                </geometry>
-                <origin xyz="0 0 0" rpy="1.5708 3.1416 3.1416"/>
-            </visual>
-            <collision>
-                <geometry>
-                    <mesh filename="package://sara_description/meshes/bras_haut.dae" scale="0.001 0.001 0.001"/>
-                </geometry>
-                <origin xyz="0 0 0" rpy="1.5708 3.1416 3.1416"/>
-            </collision>
-        </link>
-        <joint name="${name}_lower_joint" type="revolute">
-            <parent link="${name}_upper_link"/>
-            <child link="${name}_lower_link"/>
-            <limit effort="1000.0" lower="-2.14" upper="1.00" velocity="0.5"/>
-            <origin xyz="-0.085 0 0" rpy="1.5708 0 1.5708" />
-            <axis xyz="0 0 1" />
-        </joint>
-    </xacro:macro>
+   <xacro:include filename="$(find sara_description)/urdf/shoulder_v1/shoulder.gazebo.xacro" />
+   <xacro:macro name="sara_shoulder_v1" params="name parent">
+      <!-- Link and joint to raise arm at shoulder level -->
+      <link name="${name}_raise_link">
+         <visual>
+            <geometry>
+               <mesh filename="package://sara_description/meshes/epaule.dae" scale="0.001 0.001 0.001"/>
+            </geometry>
+            <origin xyz="0 0 0" rpy="0 3.1416 0"/>
+         </visual>
+         <collision>
+            <geometry>
+               <mesh filename="package://sara_description/meshes/epaule.dae" scale="0.001 0.001 0.001"/>
+            </geometry>
+            <origin xyz="0 0 0" rpy="0 3.1416 0"/>
+         </collision>
+      </link>
+      <joint name="${name}_raise_joint" type="revolute">
+         <parent link="${parent}_link"/>
+         <child link="${name}_raise_link"/>
+         <limit effort="1000.0" lower="-0.18" upper="1.21" velocity="0.5"/>
+         <origin xyz="0.008948 -0.145 0.155" rpy="0 -1.57 0" />
+         <axis xyz="0 0 1" />
+      </joint>
+      <!-- Link and joint to rotate the upper part of the arm at shoulder level -->
+      <link name="${name}_upper_link">
+         <visual>
+            <geometry>
+               <mesh filename="package://sara_description/meshes/epaule.dae" scale="0.001 0.001 0.001"/>
+            </geometry>
+            <origin xyz="0 0 0" rpy="3.1416 0 1.5708"/>
+         </visual>
+         <collision>
+            <geometry>
+               <mesh filename="package://sara_description/meshes/epaule.dae" scale="0.001 0.001 0.001"/>
+            </geometry>
+            <origin xyz="0 0 0" rpy="3.1416 0 1.5708"/>
+         </collision>
+      </link>
+      <joint name="${name}_upper_joint" type="revolute">
+         <parent link="${name}_raise_link"/>
+         <child link="${name}_upper_link"/>
+         <limit effort="1000.0" lower="-3.29" upper="0.37" velocity="0.5"/>
+         <origin xyz="0 -0.085 0" rpy="-1.57 0 0" />
+         <axis xyz="0 0 1" />
+      </joint>
+      <!-- Link and joint to rotate the lower part of the arm at shoulder level -->
+      <link name="${name}_lower_link">
+         <visual>
+            <geometry>
+               <mesh filename="package://sara_description/meshes/bras_haut.dae" scale="0.001 0.001 0.001"/>
+            </geometry>
+            <origin xyz="0 0 0" rpy="1.5708 3.1416 3.1416"/>
+         </visual>
+         <collision>
+            <geometry>
+               <mesh filename="package://sara_description/meshes/bras_haut.dae" scale="0.001 0.001 0.001"/>
+            </geometry>
+            <origin xyz="0 0 0" rpy="1.5708 3.1416 3.1416"/>
+         </collision>
+      </link>
+      <joint name="${name}_lower_joint" type="revolute">
+         <parent link="${name}_upper_link"/>
+         <child link="${name}_lower_link"/>
+         <limit effort="1000.0" lower="-2.14" upper="1.00" velocity="0.5"/>
+         <origin xyz="-0.085 0 0" rpy="1.5708 0 1.5708" />
+         <axis xyz="0 0 1" />
+      </joint>
+      <xacro:sara_shoulder_gazebo_v1 />
+   </xacro:macro>
 </robot>

File: sara_description/urdf/torso_v1/torso.urdf.xacro (robot description, xacro)
@@ -1,4 +1,5 @@
 <?xml version="1.0"?>
 <robot xmlns:xacro="http://ros.org/wiki/xacro" >
+   <xacro:include filename="$(find sara_description)/urdf/torso_v1/torso.gazebo.xacro" />
    <xacro:macro name="sara_torso_v1" params="name parent">
       <link name="${name}_link">
@@ -24,4 +25,5 @@
          </inertial>
       </link>
+      <xacro:sara_torso_gazebo_v1 />
    </xacro:macro>
 </robot>

Commit message: Wrist in the URDF

File: sara_description/urdf/arm_v1/arm.urdf.xacro (robot description, xacro)
@@ -4,4 +4,11 @@
    <xacro:macro name="sara_arm_v1" params="name parent end_effector">
        <xacro:sara_arm_gazebo_v1 name="${name}" parent="${parent}"/>
+       <joint name="${parent}_${name}_joint" type="revolute">
+          <parent link="${parent}_link"/>
+          <child link="${name}_clavicular_link"/>
+          <limit effort="1000.0" lower="-0.18" upper="1.21" velocity="0.5"/>
+          <origin xyz="0.008948 -0.145 0.155" rpy="0 -1.57 0" />
+          <axis xyz="0 0 1" />
+       </joint>
        <!-- Link and joint to raise arm at shoulder level -->
       <link name="${name}_clavicular_link">
@@ -21,31 +28,4 @@
             <mass value="1" />
             <origin xyz="0 0 0" rpy="0 3.1416 0" />
-            <inertia ixx="0.001" ixy="0" ixz="0" iyy="0.001" iyz="0" izz="0.001" />
-        </inertial>
-      </link>
-      <joint name="${parent}_${name}_joint" type="revolute">
-         <parent link="${parent}_link"/>
-         <child link="${name}_clavicular_link"/>
-         <limit effort="1000.0" lower="-0.18" upper="1.21" velocity="0.5"/>
-         <origin xyz="0.008948 -0.145 0.155" rpy="0 -1.57 0" />
-         <axis xyz="0 0 1" />
-      </joint>
-      <!-- Link and joint to rotate the upper part of the arm at shoulder level -->
-      <link name="${name}_fix_upper_link">
-         <visual>
-            <geometry>
-               <mesh filename="package://sara_description/meshes/epaule.dae" scale="0.001 0.001 0.001"/>
-            </geometry>
-            <origin xyz="0 0 0" rpy="3.1416 0 1.5708"/>
-         </visual>
-         <collision>
-            <geometry>
-               <mesh filename="package://sara_description/meshes/epaule.dae" scale="0.001 0.001 0.001"/>
-            </geometry>
-            <origin xyz="0 0 0" rpy="3.1416 0 1.5708"/>
-         </collision>
-         <inertial>
-            <mass value="1" />
-            <origin xyz="0 0 0" rpy="3.1416 0 1.5708" />
             <inertia ixx="0.001" ixy="0" ixz="0" iyy="0.001" iyz="0" izz="0.001" />
         </inertial>
@@ -58,21 +38,21 @@
          <axis xyz="0 0 1" />
       </joint>
-      <!-- Link and joint to rotate the lower part of the arm at shoulder level -->
-      <link name="${name}_rot_upper_link">
-         <visual>
-            <geometry>
-               <mesh filename="package://sara_description/meshes/bras_haut.dae" scale="0.001 0.001 0.001"/>
-            </geometry>
-            <origin xyz="0 0 0" rpy="1.5708 3.1416 3.1416"/>
-         </visual>
-         <collision>
-            <geometry>
-               <mesh filename="package://sara_description/meshes/bras_haut.dae" scale="0.001 0.001 0.001"/>
-            </geometry>
-            <origin xyz="0 0 0" rpy="1.5708 3.1416 3.1416"/>
-         </collision>
-        <inertial>
-            <mass value="1" />
-            <origin xyz="0 0 0" rpy="1.5708 3.1416 3.1416" />
+      <!-- Link and joint to rotate the upper part of the arm at shoulder level -->
+      <link name="${name}_fix_upper_link">
+         <visual>
+            <geometry>
+               <mesh filename="package://sara_description/meshes/epaule.dae" scale="0.001 0.001 0.001"/>
+            </geometry>
+            <origin xyz="0 0 0" rpy="3.1416 0 1.5708"/>
+         </visual>
+         <collision>
+            <geometry>
+               <mesh filename="package://sara_description/meshes/epaule.dae" scale="0.001 0.001 0.001"/>
+            </geometry>
+            <origin xyz="0 0 0" rpy="3.1416 0 1.5708"/>
+         </collision>
+         <inertial>
+            <mass value="1" />
+            <origin xyz="0 0 0" rpy="3.1416 0 1.5708" />
             <inertia ixx="0.001" ixy="0" ixz="0" iyy="0.001" iyz="0" izz="0.001" />
         </inertial>
@@ -85,24 +65,24 @@
          <axis xyz="0 0 1" />
       </joint>
-       <!-- Link and joint to raise arm at elbow level -->
-      <link name="${name}_fix_lower_link">
-         <visual>
-            <geometry>
-               <mesh filename="package://sara_description/meshes/coude.dae" scale="0.001 0.001 0.001"/>
-            </geometry>
-            <origin xyz="0 0 -0.0005" rpy="3.1416 0 0"/>
-         </visual>
-         <collision>
-            <geometry>
-               <mesh filename="package://sara_description/meshes/coude.dae" scale="0.001 0.001 0.001"/>
-            </geometry>
-            <origin xyz="0 0 -0.0005" rpy="3.1416 0 0"/>
-         </collision>
-         <inertial>
-            <mass value="1" />
-            <origin xyz="0 0 0" rpy="0 3.1416 0" />
-            <inertia ixx="0.001" ixy="0" ixz="0" iyy="0.001" iyz="0" izz="0.001" />
-        </inertial>
-     </link>
+      <!-- Link and joint to rotate the lower part of the arm at shoulder level -->
+      <link name="${name}_rot_upper_link">
+         <visual>
+            <geometry>
+               <mesh filename="package://sara_description/meshes/bras_haut.dae" scale="0.001 0.001 0.001"/>
+            </geometry>
+            <origin xyz="0 0 0" rpy="1.5708 3.1416 3.1416"/>
+         </visual>
+         <collision>
+            <geometry>
+               <mesh filename="package://sara_description/meshes/bras_haut.dae" scale="0.001 0.001 0.001"/>
+            </geometry>
+            <origin xyz="0 0 0" rpy="1.5708 3.1416 3.1416"/>
+         </collision>
+        <inertial>
+            <mass value="1" />
+            <origin xyz="0 0 0" rpy="1.5708 3.1416 3.1416" />
+            <inertia ixx="0.001" ixy="0" ixz="0" iyy="0.001" iyz="0" izz="0.001" />
+        </inertial>
+      </link>
       <joint name="${name}_elbow_joint" type="revolute">
          <parent link="${name}_rot_upper_link"/>
@@ -112,4 +92,31 @@
          <axis xyz="0 0 1" />
       </joint>
+       <!-- Link and joint to raise arm at elbow level -->
+      <link name="${name}_fix_lower_link">
+         <visual>
+            <geometry>
+               <mesh filename="package://sara_description/meshes/coude.dae" scale="0.001 0.001 0.001"/>
+            </geometry>
+            <origin xyz="0 0 -0.0005" rpy="3.1416 0 0"/>
+         </visual>
+         <collision>
+            <geometry>
+               <mesh filename="package://sara_description/meshes/coude.dae" scale="0.001 0.001 0.001"/>
+            </geometry>
+            <origin xyz="0 0 -0.0005" rpy="3.1416 0 0"/>
+         </collision>
+         <inertial>
+            <mass value="1" />
+            <origin xyz="0 0 0" rpy="0 3.1416 0" />
+            <inertia ixx="0.001" ixy="0" ixz="0" iyy="0.001" iyz="0" izz="0.001" />
+        </inertial>
+     </link>
+     <joint name="${name}_rot_wrist_joint" type="revolute">
+        <parent link="${name}_fix_lower_link"/>
+        <child link="${name}_rot_lower_link"/>
+        <limit effort="1000.0" lower="-3.1416" upper="3.1416" velocity="0.5"/>
+        <origin xyz="0 0.0945 0" rpy="1.5708 -1.5708 0" />
+        <axis xyz="0 0 1" />
+    </joint>
       <!-- Link and joint to rotate arm at elbow level -->
       <link name="${name}_rot_lower_link">
@@ -132,13 +139,48 @@
         </inertial>
      </link>
-      <joint name="${name}_rot_wrist_joint" type="revolute">
-         <parent link="${name}_fix_lower_link"/>
-         <child link="${name}_rot_lower_link"/>
+      <joint name="${name}_abc_joint" type="revolute">
+         <parent link="${name}_rot_lower_link"/>
+         <child link="${name}_high_wrist_joint"/>
          <limit effort="1000.0" lower="-3.1416" upper="3.1416" velocity="0.5"/>
          <origin xyz="0 0.0945 0" rpy="1.5708 -1.5708 0" />
          <axis xyz="0 0 1" />
      </joint>
+     <link name="${name}_high_wrist_joint">
+          <visual>
+              <geometry>
+                  <mesh filename="package://sara_description/meshes/poignet_haut.STL" scale="0.001 0.001 0.001"/>
+              </geometry>
+              <origin xyz="0 0 0" rpy="-1.5708 0 -1.5708"/>
+          </visual>
+          <collision>
+             <geometry>
+                <mesh filename="package://sara_description/meshes/poignet_haut.STL" scale="0.001 0.001 0.001"/>
+             </geometry>
+             <origin xyz="0 0 0" rpy="-1.5708 0 -1.5708"/>
+          </collision>
+     </link>
+     <joint name="${name}_wrist_joint" type="revolute">
+        <parent link="${name}_high_wrist_joint"/>
+        <child link="${name}_low_wrist_joint"/>
+        <limit effort="1000.0" lower="-3.1416" upper="3.1416" velocity="0.5"/>
+        <origin xyz="0 0.0945 0" rpy="1.5708 -1.5708 0" />
+        <axis xyz="0 0 1" />
+     </joint>
+     <link name="${name}_low_wrist_joint">
+          <visual>
+              <geometry>
+                  <mesh filename="package://sara_description/meshes/poignet_bas.STL" scale="0.001 0.001 0.001"/>
+              </geometry>
+              <origin xyz="0 0 0" rpy="-1.5708 0 -1.5708"/>
+          </visual>
+          <collision>
+             <geometry>
+                <mesh filename="package://sara_description/meshes/poignet_bas.STL" scale="0.001 0.001 0.001"/>
+             </geometry>
+             <origin xyz="0 0 0" rpy="-1.5708 0 -1.5708"/>
+          </collision>
+     </link>
       <joint name="${name}_end_effector_joint" type="fixed">
-         <parent link="${name}_rot_lower_link"/>
+         <parent link="${name}_low_wrist_joint"/>
          <child link="${end_effector}_link"/>
          <limit effort="1000.0" lower="-0.26" upper="0.26" velocity="0.5" />

Commit message: Save Commit

File: sara_description/urdf/arm_v1/arm.urdf.xacro (robot description, xacro)
@@ -123,27 +123,28 @@
          <visual>
             <geometry>
-               <mesh filename="package://sara_description/meshes/avant-bras.dae" scale="0.001 0.001 0.001"/>
-            </geometry>
-            <origin xyz="0 0 0" rpy="-1.5708 0 -1.5708"/>
-         </visual>
-         <collision>
-            <geometry>
-               <mesh filename="package://sara_description/meshes/avant-bras.dae" scale="0.001 0.001 0.001"/>
-            </geometry>
-            <origin xyz="0 0 0" rpy="-1.5708 0 -1.5708"/>
+               <mesh filename="package://sara_description/meshes/avant-bras.STL" scale="0.001 0.001 0.001"/>
+            </geometry>
+            <origin xyz="-0.0338 0.0338 0" rpy="-1.5708 0 -1.5708" />
+         </visual>
+         <collision>
+            <geometry>
+               <mesh filename="package://sara_description/meshes/avant-bras.STL" scale="0.001 0.001 0.001"/>
+            </geometry>
+            <origin xyz="-0.0676 0.0676 0" rpy="-1.5708 0 -1.5708" />
          </collision>
           <inertial>
             <mass value="1" />
-            <origin xyz="0 0 0" rpy="-1.5708 0 -1.5708" />
-            <inertia ixx="0.001" ixy="0" ixz="0" iyy="0.001" iyz="0" izz="0.001" />
-        </inertial>
-     </link>
-      <joint name="${name}_abc_joint" type="revolute">
+            <origin xyz="-0.0676 0.0676 0" rpy="-1.5708 0 -1.5708" />
+            <inertia ixx="0.001" ixy="0" ixz="0" iyy="0.001" iyz="0" izz="0.001" />
+        </inertial>
+     </link>
+      <joint name="${name}_forarm-wrist_joint" type="revolute">
          <parent link="${name}_rot_lower_link"/>
          <child link="${name}_high_wrist_joint"/>
          <limit effort="1000.0" lower="-3.1416" upper="3.1416" velocity="0.5"/>
-         <origin xyz="0 0.0945 0" rpy="1.5708 -1.5708 0" />
-         <axis xyz="0 0 1" />
+	 <origin xyz="0 0 -0.11184" rpy="1.5708 -1.5708 0" />
+         <axis xyz="0 1 0" />
      </joint>
+     <!-- First wrist joint and link | forarm to wrist -->
      <link name="${name}_high_wrist_joint">
           <visual>
@@ -151,5 +152,5 @@
                   <mesh filename="package://sara_description/meshes/poignet_haut.STL" scale="0.001 0.001 0.001"/>
               </geometry>
-              <origin xyz="0 0 0" rpy="-1.5708 0 -1.5708"/>
+              <origin xyz="0.0706 0 -0.030" rpy="1.5708 -1.5708 0"/>
           </visual>
           <collision>
@@ -164,7 +165,8 @@
         <child link="${name}_low_wrist_joint"/>
         <limit effort="1000.0" lower="-3.1416" upper="3.1416" velocity="0.5"/>
-        <origin xyz="0 0.0945 0" rpy="1.5708 -1.5708 0" />
-        <axis xyz="0 0 1" />
+        <origin xyz="-0.084642 0 0" rpy="1.5708 -1.5708 0" />
+        <axis xyz="1 0 0" />
      </joint>
+     <!-- Second wrist joint and link | wrist to Robotiq grasp -->
      <link name="${name}_low_wrist_joint">
           <visual>
@@ -172,5 +174,5 @@
                   <mesh filename="package://sara_description/meshes/poignet_bas.STL" scale="0.001 0.001 0.001"/>
               </geometry>
-              <origin xyz="0 0 0" rpy="-1.5708 0 -1.5708"/>
+              <origin xyz="0.0275 -0.084375 0" rpy="0 -1.5708 0"/>
           </visual>
           <collision>
@@ -205,5 +207,5 @@
           <parent link="${end_effector}_link" />
          <child link="grasp_link" />
-         <origin xyz="0.075 0 -0.012" rpy="3.1416 0 1.5708" />
+         <origin xyz="0.075 0 -0.012" rpy="0 0 0" />
       </joint>
    </xacro:macro>

Commit message: Right names for links | wrist parts in right places

File: sara_description/urdf/arm_v1/arm.urdf.xacro (robot description, xacro)
@@ -141,5 +141,5 @@
       <joint name="${name}_forarm-wrist_joint" type="revolute">
          <parent link="${name}_rot_lower_link"/>
-         <child link="${name}_high_wrist_joint"/>
+         <child link="${name}_high_wrist_link"/>
          <limit effort="1000.0" lower="-3.1416" upper="3.1416" velocity="0.5"/>
 	 <origin xyz="0 0 -0.11184" rpy="1.5708 -1.5708 0" />
@@ -147,10 +147,10 @@
      </joint>
      <!-- First wrist joint and link | forarm to wrist -->
-     <link name="${name}_high_wrist_joint">
+     <link name="${name}_high_wrist_link">
           <visual>
               <geometry>
                   <mesh filename="package://sara_description/meshes/poignet_haut.STL" scale="0.001 0.001 0.001"/>
               </geometry>
-              <origin xyz="0.0706 0 -0.030" rpy="1.5708 -1.5708 0"/>
+              <origin xyz="0.0706 0.0283 -0.030" rpy="1.5708 -1.5708 0"/>
           </visual>
           <collision>
@@ -162,6 +162,6 @@
      </link>
      <joint name="${name}_wrist_joint" type="revolute">
-        <parent link="${name}_high_wrist_joint"/>
-        <child link="${name}_low_wrist_joint"/>
+        <parent link="${name}_high_wrist_link"/>
+        <child link="${name}_low_wrist_link"/>
         <limit effort="1000.0" lower="-3.1416" upper="3.1416" velocity="0.5"/>
         <origin xyz="-0.084642 0 0" rpy="1.5708 -1.5708 0" />
@@ -169,10 +169,10 @@
      </joint>
      <!-- Second wrist joint and link | wrist to Robotiq grasp -->
-     <link name="${name}_low_wrist_joint">
+     <link name="${name}_low_wrist_link">
           <visual>
               <geometry>
                   <mesh filename="package://sara_description/meshes/poignet_bas.STL" scale="0.001 0.001 0.001"/>
               </geometry>
-              <origin xyz="0.0275 -0.084375 0" rpy="0 -1.5708 0"/>
+              <origin xyz="0.0275 -0.09839 -0.0305448" rpy="0 -1.5708 0"/>
           </visual>
           <collision>
@@ -184,5 +184,5 @@
      </link>
       <joint name="${name}_end_effector_joint" type="fixed">
-         <parent link="${name}_low_wrist_joint"/>
+         <parent link="${name}_low_wrist_link"/>
          <child link="${end_effector}_link"/>
          <limit effort="1000.0" lower="-0.26" upper="0.26" velocity="0.5" />
