Commit message: Fixed grasp | Good rotation of all components except socket

File: sara_description/urdf/arm_v1/arm.urdf.xacro (robot description, xacro)
@@ -139,12 +139,11 @@
         </inertial>
      </link>
-      <joint name="${name}_forarm-wrist_joint" type="revolute">
-         <parent link="${name}_rot_lower_link"/>
-         <child link="${name}_high_wrist_link"/>
-         <limit effort="1000.0" lower="-3.1416" upper="3.1416" velocity="0.5"/>
-	 <origin xyz="0 0 -0.11184" rpy="1.5708 -1.5708 0" />
-         <axis xyz="0 1 0" />
-     </joint>
-     <!-- First wrist joint and link | forarm to wrist -->
+     <joint name="${name}_forarm-wrist_joint" type="fixed">
+        <parent link="${name}_rot_lower_link"/>
+        <child link="${name}_high_wrist_link"/>
+        <limit effort="1000.0" lower="-3.1416" upper="3.1416" velocity="0.5"/>
+        <origin xyz="0 0 -0.11184" rpy="1.5708 -1.5708 0" />
+        <axis xyz="0 1 0" />
+    </joint>
      <link name="${name}_high_wrist_link">
           <visual>
@@ -161,12 +160,11 @@
           </collision>
      </link>
-     <joint name="${name}_wrist_joint" type="revolute">
+     <joint name="${name}_high_low_wrist_joint" type="revolute">
         <parent link="${name}_high_wrist_link"/>
         <child link="${name}_low_wrist_link"/>
         <limit effort="1000.0" lower="-3.1416" upper="3.1416" velocity="0.5"/>
-        <origin xyz="-0.084642 0 0" rpy="1.5708 -1.5708 0" />
-        <axis xyz="1 0 0" />
-     </joint>
-     <!-- Second wrist joint and link | wrist to Robotiq grasp -->
+        <origin xyz="0 0 0" rpy="1.5708 -1.5708 0" />
+        <axis xyz="0 0 1" />
+    </joint>
      <link name="${name}_low_wrist_link">
           <visual>
@@ -174,5 +172,5 @@
                   <mesh filename="package://sara_description/meshes/poignet_bas.STL" scale="0.001 0.001 0.001"/>
               </geometry>
-              <origin xyz="0.0275 -0.09839 -0.0305448" rpy="0 -1.5708 0"/>
+              <origin xyz="0.0257591 -0.014017 -0.028925" rpy="0 -1.5708 0"/>
           </visual>
           <collision>
@@ -183,6 +181,21 @@
           </collision>
      </link>
+          <joint name="${name}_low_wrist_grasp_socket_joint" type="revolute">
+             <parent link="${name}_low_wrist_link"/>
+             <child link="${name}_socket_link"/>
+             <limit effort="1000.0" lower="-3.1416" upper="3.1416" velocity="0.5"/>
+             <origin xyz="0 0 0" rpy="1.5708 0 0" />
+             <axis xyz="1 0 0" />
+          </joint>
+      <link name="${name}_socket_link">
+      <visual>
+          <geometry>
+              <mesh filename="package://sara_description/meshes/attache-pince.STL" scale="0.001 0.001 0.001"/>
+          </geometry>
+          <origin xyz="0 0 0" rpy="0 0 0"/>
+      </visual>
+      </link>
       <joint name="${name}_end_effector_joint" type="fixed">
-         <parent link="${name}_low_wrist_link"/>
+         <parent link="${name}_socket_link"/>
          <child link="${end_effector}_link"/>
          <limit effort="1000.0" lower="-0.26" upper="0.26" velocity="0.5" />

Commit message: Working URDF | grasp in the right place

File: sara_description/urdf/arm_v1/arm.urdf.xacro (robot description, xacro)
@@ -126,4 +126,5 @@
             </geometry>
             <origin xyz="-0.0338 0.0338 0" rpy="-1.5708 0 -1.5708" />
+             <color rgba="0 0 1 .06"/>
          </visual>
          <collision>
@@ -152,4 +153,5 @@
               </geometry>
               <origin xyz="0.0706 0.0283 -0.030" rpy="1.5708 -1.5708 0"/>
+              <color rgba="0 0 1 .06"/>
           </visual>
           <collision>
@@ -172,5 +174,6 @@
                   <mesh filename="package://sara_description/meshes/poignet_bas.STL" scale="0.001 0.001 0.001"/>
               </geometry>
-              <origin xyz="0.0257591 -0.014017 -0.028925" rpy="0 -1.5708 0"/>
+              <origin xyz="-0.02575  -0.01375 0.0305448" rpy=" 0 1.5708 0"/>
+              <color rgba="0 0 1 .06"/>
           </visual>
           <collision>
@@ -178,5 +181,5 @@
                 <mesh filename="package://sara_description/meshes/poignet_bas.STL" scale="0.001 0.001 0.001"/>
              </geometry>
-             <origin xyz="0 0 0" rpy="-1.5708 0 -1.5708"/>
+             <origin xyz="0 0 0" rpy="0 0 0 "/>
           </collision>
      </link>
@@ -185,5 +188,5 @@
              <child link="${name}_socket_link"/>
              <limit effort="1000.0" lower="-3.1416" upper="3.1416" velocity="0.5"/>
-             <origin xyz="0 0 0" rpy="1.5708 0 0" />
+             <origin xyz="0 0.084375 0" rpy="1.5708 0 0" />
              <axis xyz="1 0 0" />
           </joint>
@@ -193,32 +196,33 @@
               <mesh filename="package://sara_description/meshes/attache-pince.STL" scale="0.001 0.001 0.001"/>
           </geometry>
-          <origin xyz="0 0 0" rpy="0 0 0"/>
+          <origin xyz="0.028925 -0.025 -0.0362070" rpy="0 0 1.5708"/>
+          <color rgba="0 0 1 .06"/>
       </visual>
       </link>
       <joint name="${name}_end_effector_joint" type="fixed">
-         <parent link="${name}_socket_link"/>
-         <child link="${end_effector}_link"/>
-         <limit effort="1000.0" lower="-0.26" upper="0.26" velocity="0.5" />
-         <axis xyz="0 1 0"/>
-         <origin xyz="0 -0.004 -0.10624" rpy="0 1.5708 1.5708"/>
-      </joint>
-      <!-- Link and joint for target (grasp) -->
-      <link name="grasp_link" >
-         <visual>
-            <geometry>
-               <sphere radius="0.01" />
-            </geometry>
-            <origin xyz="0 0.05 0" rpy="0 0 0" />
-         </visual>
-         <inertial>
-            <mass value="0" />
-            <origin xyz="0 0 0" rpy="0 0 0" />
-            <inertia ixx="0.001" ixy="0" ixz="0" iyy="0.001" iyz="0" izz="0.001" />
-        </inertial>
-      </link>
-      <joint name="grasp_joint" type="fixed" >
-          <parent link="${end_effector}_link" />
-         <child link="grasp_link" />
-         <origin xyz="0.075 0 -0.012" rpy="0 0 0" />
+               <parent link="${name}_socket_link"/>
+               <child link="${end_effector}_link"/>
+               <limit effort="1000.0" lower="-0.26" upper="0.26" velocity="0.5" />
+               <axis xyz="0 1 0"/>
+               <origin xyz="0 0 -0.0298927" rpy="0 1.5708 0"/>
+            </joint>
+            <!-- Link and joint for target (grasp) -->
+            <link name="grasp_link" >
+               <visual>
+                  <geometry>
+                     <sphere radius="0.01" />
+                  </geometry>
+                  <origin xyz="0 0.05 0" rpy="0 0 0" />
+               </visual>
+               <inertial>
+                  <mass value="0" />
+                  <origin xyz="0 0 0" rpy="0 0 0" />
+                  <inertia ixx="0.001" ixy="0" ixz="0" iyy="0.001" iyz="0" izz="0.001" />
+              </inertial>
+            </link>
+            <joint name="grasp_joint" type="fixed" >
+                <parent link="${end_effector}_link" />
+               <child link="grasp_link" />
+               <origin xyz="0.075 0 -0.012" rpy="3.1416 0 1.5708" />
       </joint>
    </xacro:macro>

Commit message: Deletion of DAE files in /meshes | Calling STL Files instead

File: sara_description/urdf/arm_v1/arm.urdf.xacro (robot description, xacro)
@@ -15,5 +15,5 @@
          <visual>
             <geometry>
-               <mesh filename="package://sara_description/meshes/epaule.dae" scale="0.001 0.001 0.001"/>
+               <mesh filename="package://sara_description/meshes/epaule.STL" scale="0.001 0.001 0.001"/>
             </geometry>
             <origin xyz="0 0 0" rpy="0 3.1416 0"/>
@@ -21,5 +21,5 @@
          <collision>
             <geometry>
-               <mesh filename="package://sara_description/meshes/epaule.dae" scale="0.001 0.001 0.001"/>
+               <mesh filename="package://sara_description/meshes/epaule.STL" scale="0.001 0.001 0.001"/>
             </geometry>
             <origin xyz="0 0 0" rpy="0 3.1416 0"/>
@@ -42,5 +42,5 @@
          <visual>
             <geometry>
-               <mesh filename="package://sara_description/meshes/epaule.dae" scale="0.001 0.001 0.001"/>
+               <mesh filename="package://sara_description/meshes/epaule.STL" scale="0.001 0.001 0.001"/>
             </geometry>
             <origin xyz="0 0 0" rpy="3.1416 0 1.5708"/>
@@ -48,5 +48,5 @@
          <collision>
             <geometry>
-               <mesh filename="package://sara_description/meshes/epaule.dae" scale="0.001 0.001 0.001"/>
+               <mesh filename="package://sara_description/meshes/epaule.STL" scale="0.001 0.001 0.001"/>
             </geometry>
             <origin xyz="0 0 0" rpy="3.1416 0 1.5708"/>
@@ -69,5 +69,5 @@
          <visual>
             <geometry>
-               <mesh filename="package://sara_description/meshes/bras_haut.dae" scale="0.001 0.001 0.001"/>
+               <mesh filename="package://sara_description/meshes/bras_haut.STL" scale="0.001 0.001 0.001"/>
             </geometry>
             <origin xyz="0 0 0" rpy="1.5708 3.1416 3.1416"/>
@@ -75,5 +75,5 @@
          <collision>
             <geometry>
-               <mesh filename="package://sara_description/meshes/bras_haut.dae" scale="0.001 0.001 0.001"/>
+               <mesh filename="package://sara_description/meshes/bras_haut.STL" scale="0.001 0.001 0.001"/>
             </geometry>
             <origin xyz="0 0 0" rpy="1.5708 3.1416 3.1416"/>
@@ -96,5 +96,5 @@
          <visual>
             <geometry>
-               <mesh filename="package://sara_description/meshes/coude.dae" scale="0.001 0.001 0.001"/>
+               <mesh filename="package://sara_description/meshes/coude.STL" scale="0.001 0.001 0.001"/>
             </geometry>
             <origin xyz="0 0 -0.0005" rpy="3.1416 0 0"/>
@@ -102,5 +102,5 @@
          <collision>
             <geometry>
-               <mesh filename="package://sara_description/meshes/coude.dae" scale="0.001 0.001 0.001"/>
+               <mesh filename="package://sara_description/meshes/coude.STL" scale="0.001 0.001 0.001"/>
             </geometry>
             <origin xyz="0 0 -0.0005" rpy="3.1416 0 0"/>
@@ -205,5 +205,5 @@
                <limit effort="1000.0" lower="-0.26" upper="0.26" velocity="0.5" />
                <axis xyz="0 1 0"/>
-               <origin xyz="0 0 -0.0298927" rpy="0 1.5708 0"/>
+               <origin xyz="0 0 -0.02989" rpy="0 1.5708 0"/>
             </joint>
             <!-- Link and joint for target (grasp) -->

File: sara_description/urdf/head_v1/head.urdf.xacro (robot description, xacro)
@@ -7,5 +7,5 @@
          <visual>
             <geometry>
-               <mesh filename="package://sara_description/meshes/tete.dae" scale="0.001 0.001 0.001" />
+               <mesh filename="package://sara_description/meshes/tete.STL" scale="0.001 0.001 0.001" />
             </geometry>
             <origin xyz="0 0 0" rpy="1.5708 -1.5708 1.5708" />
@@ -13,5 +13,5 @@
          <collision>
             <geometry>
-               <mesh filename="package://sara_description/meshes/tete.dae" scale="0.001 0.001 0.001" />
+               <mesh filename="package://sara_description/meshes/tete.STL" scale="0.001 0.001 0.001" />
             </geometry>
             <origin xyz="0 0 0" rpy="1.5708 -1.5708 1.5708" />
@@ -57,5 +57,5 @@
          <visual>
             <geometry>
-               <mesh filename="package://sara_description/meshes/xtion.dae" scale="0.001 0.001 0.001"/>
+               <mesh filename="package://sara_description/meshes/xtion.STL" scale="0.001 0.001 0.001"/>
             </geometry>
             <origin xyz="0 0 0" rpy="1.5708 0 1.5708"/>

File: sara_description/urdf/neck_v1/neck.urdf.xacro (robot description, xacro)
@@ -7,5 +7,5 @@
          <visual>
             <geometry>
-               <mesh filename="package://sara_description/meshes/cou.dae" scale="0.001 0.001 0.001"/>
+               <mesh filename="package://sara_description/meshes/cou.STL" scale="0.001 0.001 0.001"/>
             </geometry>
             <origin xyz="0 0 0" rpy="1.5708 0 1.5708"/>

File: sara_description/urdf/torso_v1/torso.urdf.xacro (robot description, xacro)
@@ -7,5 +7,5 @@
          <visual>
             <geometry>
-               <mesh filename="package://sara_description/meshes/torse.dae" scale="0.001 0.001 0.001"/>
+               <mesh filename="package://sara_description/meshes/torse.STL" scale="0.001 0.001 0.001"/>
             </geometry>
             <origin xyz="0 0 0" rpy="1.5708 0 1.5708"/>
@@ -16,5 +16,5 @@
          <collision>
             <geometry>
-               <mesh filename="package://sara_description/meshes/torse.dae" scale="0.001 0.001 0.001"/>
+               <mesh filename="package://sara_description/meshes/torse.STL" scale="0.001 0.001 0.001"/>
             </geometry>
             <origin xyz="0 0 0" rpy="1.5708 0 1.5708"/>

Commit message: Added kinect in the URDF

File: sara_description/urdf/arm_v1/arm.urdf.xacro (robot description, xacro)
@@ -8,5 +8,5 @@
           <child link="${name}_clavicular_link"/>
           <limit effort="1000.0" lower="-0.18" upper="1.21" velocity="0.5"/>
-          <origin xyz="0.008948 -0.145 0.155" rpy="0 -1.57 0" />
+          <origin xyz="0 -0.145 0.189" rpy="0 -1.57 0" />
           <axis xyz="0 0 1" />
        </joint>
@@ -18,4 +18,7 @@
             </geometry>
             <origin xyz="0 0 0" rpy="0 3.1416 0"/>
+            <material name="black">
+               <color rgba="0.12 0.12 0.12 1"/>
+            </material>
          </visual>
          <collision>
@@ -45,4 +48,7 @@
             </geometry>
             <origin xyz="0 0 0" rpy="3.1416 0 1.5708"/>
+            <material name="black">
+               <color rgba="0.12 0.12 0.12 1"/>
+            </material>
          </visual>
          <collision>
@@ -72,4 +78,7 @@
             </geometry>
             <origin xyz="0 0 0" rpy="1.5708 3.1416 3.1416"/>
+            <material name="black">
+               <color rgba="0.12 0.12 0.12 1"/>
+            </material>
          </visual>
          <collision>
@@ -99,4 +108,7 @@
             </geometry>
             <origin xyz="0 0 -0.0005" rpy="3.1416 0 0"/>
+            <material name="black">
+               <color rgba="0.12 0.12 0.12 1"/>
+            </material>
          </visual>
          <collision>
@@ -126,5 +138,7 @@
             </geometry>
             <origin xyz="-0.0338 0.0338 0" rpy="-1.5708 0 -1.5708" />
-             <color rgba="0 0 1 .06"/>
+            <material name="black">
+               <color rgba="0.12 0.12 0.12 1"/>
+            </material>
          </visual>
          <collision>
@@ -153,4 +167,6 @@
               </geometry>
               <origin xyz="0.0706 0.0283 -0.030" rpy="1.5708 -1.5708 0"/>
+              <material name="black">
+              </material>
               <color rgba="0 0 1 .06"/>
           </visual>
@@ -175,5 +191,7 @@
               </geometry>
               <origin xyz="-0.02575  -0.01375 0.0305448" rpy=" 0 1.5708 0"/>
-              <color rgba="0 0 1 .06"/>
+              <material name="black">
+                 <color rgba="0.12 0.12 0.12 1"/>
+              </material>
           </visual>
           <collision>
@@ -197,5 +215,7 @@
           </geometry>
           <origin xyz="0.028925 -0.025 -0.0362070" rpy="0 0 1.5708"/>
-          <color rgba="0 0 1 .06"/>
+          <material name="black">
+             <color rgba="0.12 0.12 0.12 1"/>
+          </material>
       </visual>
       </link>

File: sara_description/urdf/base_v1/base.urdf.xacro (robot description, xacro)
@@ -9,5 +9,5 @@
             <mesh filename="package://sara_description/meshes/base.STL" scale="0.001 0.001 0.001"/>
          </geometry>
-         <origin xyz="0.295 -0.250 0.85635" rpy="-1.57 0 1.57"/>
+         <origin xyz="0.300 -0.250 0.85635" rpy="-1.57 0 1.57"/>
          <material name="black">
                <color rgba="0.12 0.12 0.12 1"/>

File: sara_description/urdf/head_v1/head.urdf.xacro (robot description, xacro)
@@ -10,4 +10,7 @@
             </geometry>
             <origin xyz="0 0 0" rpy="1.5708 -1.5708 1.5708" />
+            <material name="blue">
+                <color rgba="0.06 0.06 1 1"/>
+            </material>
          </visual>
          <collision>

File: sara_description/urdf/neck_v1/neck.urdf.xacro (robot description, xacro)
@@ -10,4 +10,7 @@
             </geometry>
             <origin xyz="0 0 0" rpy="1.5708 0 1.5708"/>
+            <material name="blue">
+                <color rgba="0.06 0.06 1 1"/>
+            </material>
          </visual>
          <inertial>
@@ -22,5 +25,5 @@
          <limit effort="1000.0" lower="-1.22173" upper="1.22173" velocity="0.5"/>
          <!-- 1mm ajoute en z (collision) -->
-         <origin xyz="0.032295 0 0.2438" rpy="0 0 0"/>
+         <origin xyz="0.032295 0 0.2777" rpy="0 0 0"/>
          <axis xyz="0 0 1"/>
       </joint>

File: sara_description/urdf/sara.urdf.xacro (robot description, xacro)
@@ -4,4 +4,5 @@
     <xacro:include filename="$(find sara_description)/urdf/torso_v1/torso.urdf.xacro"/>
     <xacro:include filename="$(find sara_description)/urdf/neck_v1/neck.urdf.xacro"/>
+    <xacro:include filename="$(find sara_description)/urdf/kinect_v1/kinect.urdf.xacro"/>
     <xacro:include filename="$(find sara_description)/urdf/head_v1/head.urdf.xacro"/>
     <xacro:include filename="$(find sara_description)/urdf/robotiq_c2_model/robotiq_c2_model_macro.xacro"/>
@@ -13,4 +14,6 @@
     <!-- Wheels -->
     <xacro:sara_wheels_v1 name="wheels" parent="base"/>
+    <!-- Kinect -->
+    <xacro:sara_kinect_v1 name="kinect" parent="base"/>
     <!-- Torso -->
     <xacro:sara_torso_v1 name="torso" parent="base"/>

File: sara_description/urdf/torso_v1/torso.urdf.xacro (robot description, xacro)
@@ -9,5 +9,5 @@
                <mesh filename="package://sara_description/meshes/torse.STL" scale="0.001 0.001 0.001"/>
             </geometry>
-            <origin xyz="0 0 0" rpy="1.5708 0 1.5708"/>
+            <origin xyz="-0.14427 -0.197233 0" rpy="1.5708 0 1.5708"/>
             <material name="black">
                <color rgba="0.12 0.12 0.12 1"/>
@@ -30,5 +30,5 @@
          <child link="${name}_link"/>
          <limit effort="1000.0" lower="0" upper="0.5" velocity="0.2"/>
-         <origin xyz="0.199974 0 0.85635" rpy="0 0 0" />
+         <origin xyz="0.177374 0 0.70531" rpy="0 0 0" />
          <axis xyz="0 0 1" />
     </joint>
