Commit message: Collisions of meshes | Changed xacro:macro name from sara_kinect_v1 to kinect2

File: sara_description/urdf/arm_v1/arm.urdf.xacro (robot description, xacro)
@@ -146,5 +146,5 @@
                <mesh filename="package://sara_description/meshes/avant-bras.STL" scale="0.001 0.001 0.001"/>
             </geometry>
-            <origin xyz="-0.0676 0.0676 0" rpy="-1.5708 0 -1.5708" />
+            <origin xyz="-0.0338 0.0338 0" rpy="-1.5708 0 -1.5708" />
          </collision>
           <inertial>
@@ -175,5 +175,5 @@
                 <mesh filename="package://sara_description/meshes/poignet_haut.STL" scale="0.001 0.001 0.001"/>
              </geometry>
-             <origin xyz="0 0 0" rpy="-1.5708 0 -1.5708"/>
+             <origin xyz="0.0706 0.0283 -0.030" rpy="1.5708 -1.5708 0"/>
           </collision>
      </link>
@@ -199,5 +199,5 @@
                 <mesh filename="package://sara_description/meshes/poignet_bas.STL" scale="0.001 0.001 0.001"/>
              </geometry>
-             <origin xyz="0 0 0" rpy="0 0 0 "/>
+             <origin xyz="-0.02575  -0.01375 0.0305448" rpy=" 0 1.5708 0"/>
           </collision>
      </link>
@@ -219,4 +219,10 @@
           </material>
       </visual>
+      <collision>
+         <geometry>
+            <mesh filename="package://sara_description/meshes/attache-pince.STL" scale="0.001 0.001 0.001"/>
+         </geometry>
+         <origin xyz="0.028925 -0.025 -0.0362070" rpy="0 0 1.5708"/>
+      </collision>
       </link>
       <joint name="${name}_end_effector_joint" type="fixed">

File: sara_description/urdf/base_v1/base.urdf.xacro (robot description, xacro)
@@ -9,5 +9,5 @@
             <mesh filename="package://sara_description/meshes/base.STL" scale="0.001 0.001 0.001"/>
          </geometry>
-         <origin xyz="0.300 -0.250 0.85635" rpy="-1.57 0 1.57"/>
+         <origin xyz="0.295 -0.250 0.85635" rpy="-1.57 0 1.57"/>
          <material name="black">
                <color rgba="0.12 0.12 0.12 1"/>

File: sara_description/urdf/head_v1/head.urdf.xacro (robot description, xacro)
@@ -65,4 +65,10 @@
             <material name="black"/>
          </visual>
+         <collision>
+            <geometry>
+               <mesh filename="package://sara_description/meshes/xtion.STL" scale="0.001 0.001 0.001"/>
+            </geometry>
+            <origin xyz="0 0 0" rpy="1.5708 0 1.5708"/>
+         </collision>
          <inertial>
             <mass value="0.5"/>

File: sara_description/urdf/kinect_v1/kinect.gazebo.xacro (robot description, xacro)
@@ -1,5 +1,5 @@
 <?xml version="1.0"?>
 <robot xmlns:xacro="http://ros.org/wiki/xacro">
-   <xacro:macro name="sara_kinect_gazebo_v1" params="name parent">
+   <xacro:macro name="kinect2_gazebo" params="name parent">
       <gazebo reference="${name}_link">
          <gravity>false</gravity>

File: sara_description/urdf/kinect_v1/kinect.urdf.xacro (robot description, xacro)
@@ -2,6 +2,6 @@
 <robot xmlns:xacro="http://ros.org/wiki/xacro" >
    <xacro:include filename="$(find sara_description)/urdf/kinect_v1/kinect.gazebo.xacro" />
-   <xacro:macro name="sara_kinect_v1" params="name parent">
-       <xacro:sara_kinect_gazebo_v1 name="${name}" parent="${parent}"/>
+   <xacro:macro name="kinect2" params="name parent">
+       <xacro:kinect2_gazebo name="${name}" parent="${parent}"/>
        <link name="${name}_link">
          <visual>
@@ -18,5 +18,5 @@
                <mesh filename="package://sara_description/meshes/kinect.STL" scale="0.001 0.001 0.001"/>
             </geometry>
-            <origin xyz="0 0 0" rpy="1.5708 0 1.5708"/>
+            <origin xyz="-0.0269875 0.1321628 0" rpy="0 0 -1.5708"/>
          </collision>
          <inertial>

File: sara_description/urdf/neck_v1/neck.urdf.xacro (robot description, xacro)
@@ -14,4 +14,10 @@
             </material>
          </visual>
+         <collision>
+            <geometry>
+               <mesh filename="package://sara_description/meshes/cou.STL" scale="0.001 0.001 0.001"/>
+            </geometry>
+            <origin xyz="0 0 0" rpy="1.5708 0 1.5708"/>
+         </collision>
          <inertial>
             <mass value="2"/>

File: sara_description/urdf/sara.urdf.xacro (robot description, xacro)
@@ -15,5 +15,5 @@
     <xacro:sara_wheels_v1 name="wheels" parent="base"/>
     <!-- Kinect -->
-    <xacro:sara_kinect_v1 name="kinect" parent="base"/>
+    <xacro:kinect2 name="kinect" parent="base"/>
     <!-- Torso -->
     <xacro:sara_torso_v1 name="torso" parent="base"/>

File: sara_description/urdf/torso_v1/torso.urdf.xacro (robot description, xacro)
@@ -18,9 +18,9 @@
                <mesh filename="package://sara_description/meshes/torse.STL" scale="0.001 0.001 0.001"/>
             </geometry>
-            <origin xyz="0 0 0" rpy="1.5708 0 1.5708"/>
+            <origin xyz="-0.14427 -0.197233 0" rpy="1.5708 0 1.5708"/>
          </collision>
          <inertial>
             <mass value="10"/>
-            <origin xyz="0 0 0" rpy="1.5708 0 1.5708"/>
+            <origin xyz="-0.14427 -0.197233 0" rpy="1.5708 0 1.5708"/>
             <inertia ixx="0.001" ixy="0" ixz="0" iyy="0.001" iyz="0" izz="0.001"/>
          </inertial>
