Commit message: updated wheel links

File: sara_description/urdf/wheels_v1/wheels.urdf.xacro (robot description, xacro)
@@ -2,6 +2,6 @@
 <robot xmlns:xacro="http://ros.org/wiki/xacro" >
    <xacro:include filename="$(find sara_description)/urdf/wheels_v1/wheels.gazebo.xacro" />
-   <!-- Wheel -->
-  <xacro:macro name="wheel" params="prefix y_reflect x_reflect x_axis_rotation">
+   <!-- Front_Wheels -->
+  <xacro:macro name="front_wheel" params="prefix y_reflect x_reflect x_axis_rotation">
       <link name="${prefix}_wheel">
           <visual>
@@ -25,10 +25,36 @@
           <child link="${prefix}_wheel"/>
           <axis xyz="0 0 1"/>
-          <origin xyz="${y_reflect * 0.230631} ${x_reflect * 0.22735} 0" rpy=" ${x_axis_rotation * 1.57079632679} 0 0"/>
+          <origin xyz="${y_reflect * 0.2056310} ${x_reflect * 0.22735} -0.06" rpy=" ${x_axis_rotation * 1.57079632679} 0 0"/>
       </joint>
    </xacro:macro>
-   <xacro:wheel prefix="front_left" y_reflect="1" x_reflect="1" x_axis_rotation="-1"/>
-   <xacro:wheel prefix="front_right" y_reflect="1" x_reflect="-1" x_axis_rotation="1"/>
-   <xacro:wheel prefix="rear_left" y_reflect="-1" x_reflect="1" x_axis_rotation="-1"/>
-   <xacro:wheel prefix="rear_right" y_reflect="-1" x_reflect="-1" x_axis_rotation="1"/>
+   <!-- rear_Wheels -->
+  <xacro:macro name="rear_wheel" params="prefix y_reflect x_reflect x_axis_rotation">
+      <link name="${prefix}_wheel">
+          <visual>
+              <geometry>
+                  <cylinder length="0.04" radius="0.15"/>
+              </geometry>
+              <origin xyz="0 0 0" rpy="0 0 0"/>
+              <material name="black">
+                  <color rgba="0 0 0 0"/>
+              </material>
+          </visual>
+          <collision>
+              <geometry>
+                  <cylinder length="0.04" radius="0.15"/>
+              </geometry>
+              <origin xyz="0 0 0" rpy="0 0 0"/>
+          </collision>
+      </link>
+      <joint name="base_to_${prefix}_wheel" type="continuous">
+          <parent link="base_link"/>
+          <child link="${prefix}_wheel"/>
+          <axis xyz="0 0 1"/>
+          <origin xyz="${y_reflect * 0.255631} ${x_reflect * 0.22735} -0.06" rpy=" ${x_axis_rotation * 1.57079632679} 0 0"/>
+      </joint>
+   </xacro:macro>
+   <xacro:front_wheel prefix="front_left" y_reflect="1" x_reflect="1" x_axis_rotation="-1"/>
+   <xacro:front_wheel prefix="front_right" y_reflect="1" x_reflect="-1" x_axis_rotation="1"/>
+   <xacro:rear_wheel prefix="rear_left" y_reflect="-1" x_reflect="1" x_axis_rotation="-1"/>
+   <xacro:rear_wheel prefix="rear_right" y_reflect="-1" x_reflect="-1" x_axis_rotation="1"/>
 </robot>

Commit message: True wheels size

File: sara_description/urdf/wheels_v1/wheels.urdf.xacro (robot description, xacro)
@@ -6,19 +6,4 @@
   <xacro:macro name="front_wheel" params="prefix y_reflect x_reflect x_axis_rotation">
       <link name="${prefix}_wheel">
-          <visual>
-              <geometry>
-                  <cylinder length="0.04" radius="0.15"/>
-              </geometry>
-              <origin xyz="0 0 0" rpy="0 0 0"/>
-              <material name="black">
-                  <color rgba="0 0 0 0"/>
-              </material>
-          </visual>
-          <collision>
-              <geometry>
-                  <cylinder length="0.04" radius="0.15"/>
-              </geometry>
-              <origin xyz="0 0 0" rpy="0 0 0"/>
-          </collision>
       </link>
       <joint name="base_to_${prefix}_wheel" type="continuous">
@@ -32,19 +17,4 @@
   <xacro:macro name="rear_wheel" params="prefix y_reflect x_reflect x_axis_rotation">
       <link name="${prefix}_wheel">
-          <visual>
-              <geometry>
-                  <cylinder length="0.04" radius="0.15"/>
-              </geometry>
-              <origin xyz="0 0 0" rpy="0 0 0"/>
-              <material name="black">
-                  <color rgba="0 0 0 0"/>
-              </material>
-          </visual>
-          <collision>
-              <geometry>
-                  <cylinder length="0.04" radius="0.15"/>
-              </geometry>
-              <origin xyz="0 0 0" rpy="0 0 0"/>
-          </collision>
       </link>
       <joint name="base_to_${prefix}_wheel" type="continuous">
