Commit message: Fixed URDF

File: sara_description/urdf/base_v1/base.urdf.xacro (robot description, xacro)
@@ -25,5 +25,5 @@
       </inertial>
     </link>
-    <joint name="spine_torso_joint" type="fixed">
+    <!--<joint name="spine_torso_joint" type="fixed">
       <parent link="spine_link"/>
       <child link="${parent}_link"/>
@@ -31,5 +31,5 @@
       <origin xyz="0 0 1.112" rpy="0 0 0" />
       <axis xyz="0 0 1" />
-    </joint>
+    </joint>-->
     <!-- Lien entre la colonne vertebrale et la base-->
     <link name="base_link">

File: sara_description/urdf/head_v1/head.urdf.xacro (robot description, xacro)
@@ -21,5 +21,5 @@
          </inertial>
       </link>
-      <link name="${parent}_dynamixel_link">
+      <link name="dynamixel_link">
          <visual>
             <geometry>
@@ -32,15 +32,17 @@
          </visual>
       </link>
-      <joint name="${name}_dynamixel_joint" type="revolute">
-         <parent link="${parent}_dynamixel_link"/>
-         <child link="${name}_link"/>
-         <limit effort="1000.0" lower="-1.00" upper="0.40" velocity="0.5"/>
-         <origin xyz="0 0 0" rpy="3.1416 0 0"/>
+     <joint name="dynamixel_joint" type="revolute">
+         <parent link="${name}_link"/>
+         <child link="dynamixel_link"/>
+         <limit effort="1000.0" lower="-1.5" upper="1.5" velocity="0.5"/>
+         <origin xyz="0 -0.054 0" rpy="3.1416 0 0"/>
          <axis xyz="0 0 1"/>
       </joint>
-      <joint name="dynamixel_neck_joint" type="fixed">
+      <joint name="${name}_neck_joint" type="revolute">
          <parent link="${parent}_link"/>
-         <child link="neck_dynamixel_link"/>
-         <origin xyz="0 0 0.0927" rpy="1.57 0 0"/>
+         <child link="${name}_link"/>
+         <limit effort="1000.0" lower="-0.40" upper="1.04" velocity="0.5"/>
+         <origin xyz="0 0 0.0927" rpy="-1.57 0 0"/>
+         <axis xyz="0 0 1" />
       </joint>
       <!-- xtion -->

File: sara_description/urdf/sara.urdf.xacro (robot description, xacro)
@@ -9,5 +9,5 @@
     <xacro:include filename="$(find sara_description)/urdf/base_v1/base.urdf.xacro"/>
     <!-- Torso -->
-    <xacro:sara_torso_v1 name="torso" parent=""/>
+    <xacro:sara_torso_v1 name="torso" parent="spine"/>
     <!-- Neck -->
     <xacro:sara_neck_v1 name="neck" parent="torso"/>
@@ -19,4 +19,4 @@
     <xacro:sara_arm_v1 name="arm" parent="shoulder"/>
     <!-- Base -->
-    <xacro:sara_base_v1 name="base" parent="torso"/>
+    <xacro:sara_base_v1 name="base" parent=""/>
 </robot>

File: sara_description/urdf/torso_v1/torso.urdf.xacro (robot description, xacro)
@@ -23,5 +23,12 @@
             <inertia ixx="0.001" ixy="0" ixz="0" iyy="0.001" iyz="0" izz="0.001"/>
          </inertial>
-      </link>
+     </link>
+     <joint name="spine_torso_joint" type="fixed">
+         <parent link="${parent}_link"/>
+         <child link="${name}_link"/>
+         <limit effort="1000.0" lower="0" upper="0.5" velocity="0.2"/>
+         <origin xyz="0 0 1.112" rpy="0 0 0" />
+         <axis xyz="0 0 1" />
+    </joint>
    </xacro:macro>
 </robot>

Commit message: first commit wheels base sara urdf

File: sara_description/urdf/base_v1/base.urdf.xacro (robot description, xacro)
@@ -8,16 +8,16 @@
       <visual>
         <geometry>
-          <box size="0.7637 0.64311 0.14"/>
+          <box size="0.71 0.52 0.095"/>
         </geometry>
-        <origin xyz="0.0 0 0.07" rpy="0 0 0"/>
+        <origin xyz="0.0 0 0.045" rpy="0 0 0"/>
         <material name="grey">
-          <color rgba="0.62 0.62 0.62 1"/>
+        <color rgba="0.62 0.62 0.62 1"/>
         </material>
       </visual>
       <visual>
         <geometry>
-          <box size="0.55 0.64311 0.57"/>
+          <box size="0.55 0.65 0.57"/>
         </geometry>
-        <origin xyz="-0.115 0 0.42" rpy="0 0 0"/>
+        <origin xyz="-0.115 0.0 1.0" rpy="0 0 0"/>
       </visual>
       <collision>
@@ -96,4 +96,32 @@
       <origin xyz="0.34 0 0.19" rpy="0 0 0" />
     </joint>
-  </xacro:macro>
+    <!-- Wheel -->
+    <xacro:macro name="wheel" params="prefix y_reflect x_reflect ">
+        <link name="${prefix}_wheel">
+            <visual>
+                <geometry>
+                    <cylinder length="0.04" radius="0.15"/>
+                </geometry>
+                <origin xyz="0 0 0" rpy="0 0 0"/>
+                <material name="black">
+                    <color rgba="0 0 0 0"/>
+                </material>
+            </visual>
+            <collision>
+                <geometry>
+                    <cylinder length="0.04" radius="0.15"/>
+                </geometry>
+                <origin xyz="0 0 0" rpy="0 0 0"/>
+            </collision>
+        </link>
+        <joint name="base_to_${prefix}_wheel" type="conti">
+            <parent link="base_link"/>
+            <child link="${prefix}_wheel"/>
+            <origin xyz="${y_reflect * } ${x_reflect * } 0" rpy/>
+        </joint>
+    </xacro:macro>
+    <xacro:wheel prefix="front_right" y_reflect="0.5" x_reflect="0.5"/>
+    <xacro:wheel prefix="front_left" y_reflect="0.5" x_reflect="0.5"/>
+    <xacro:wheel prefix="rear_right" y_reflect="0.5" x_reflect="0.5"/>
+    <xacro:wheel prefix="rear_left" y_reflect="0.5" x_reflect="0.5"/>
 </robot>

Commit message: real dimensions on wheels links

File: sara_description/urdf/base_v1/base.urdf.xacro (robot description, xacro)
@@ -4,67 +4,26 @@
   <xacro:macro name="sara_base_v1" params="name parent">
     <xacro:sara_base_gazebo_v1 name="${name}" parent="${parent}"/>
-    <!-- Lien entre la base et la colonne vertebral-->
     <link name="${name}_link">
       <visual>
-        <geometry>
-          <box size="0.71 0.52 0.095"/>
-        </geometry>
-        <origin xyz="0.0 0 0.045" rpy="0 0 0"/>
-        <material name="grey">
-        <color rgba="0.62 0.62 0.62 1"/>
-        </material>
-      </visual>
-      <visual>
-        <geometry>
-          <box size="0.55 0.65 0.57"/>
-        </geometry>
-        <origin xyz="-0.115 0.0 1.0" rpy="0 0 0"/>
+         <geometry>
+            <mesh filename="package://sara_description/meshes/base.STL" scale="0.001 0.001 0.001"/>
+         </geometry>
+         <origin xyz="0 0 0" rpy="-1.57 0 1.57"/>
       </visual>
       <collision>
-        <geometry>
-          <box size="0.7637 0.64311 0.14"/>
-        </geometry>
-        <origin xyz="0.0 0 0.07" rpy="0 0 0"/>
+         <geometry>
+            <mesh filename="package://sara_description/meshes/base.STL" scale="0.001 0.001 0.001"/>
+         </geometry>
+         <origin xyz="0 0 0" rpy="0 0 0"/>
       </collision>
-      <collision>
-        <geometry>
-          <box size="0.55 0.64311 0.57"/>
-        </geometry>
-        <origin xyz="-0.115 0 0.42" rpy="0 0 0"/>
-      </collision>
-      <inertial>
-        <mass value="10"/>
-        <origin xyz="-0.115 0 0.42" rpy="0 0 0"/>
-        <inertia ixx="0.001" ixy="0" ixz="0" iyy="0.001" iyz="0" izz="0.001"/>
-      </inertial>
     </link>
     <joint name="${name}_spine_joint" type="fixed">
       <parent link="base_link"/>
       <child link="spine_link"/>
-      <origin xyz="0.2 0 0" rpy="0 0 0" />
-      <axis xyz="0 0 1" />
+      <origin xyz="0 0 0" rpy="0 0 0" />
+      <axis xyz="0 0 0" />
     </joint>
   <!-- Lien entre le torse et la colonne vertebrale -->
     <link name="spine_link">
-      <visual>
-        <geometry>
-          <cylinder length="0.9" radius="0.04"/>
-        </geometry>
-        <origin xyz="0 0 0.49" rpy="0 0 0"/>
-        <material name="grey">
-          <color rgba="0.62 0.62 0.62 1"/>
-        </material>
-      </visual>
-      <collision>
-        <geometry>
-          <cylinder length="0.9" radius="0.07"/>
-        </geometry>
-        <origin xyz="0 0 0.49" rpy="0 0 0"/>
-      </collision>
-      <inertial>
-        <mass value="10"/>
-        <origin xyz="0 0 0.49" rpy="0 0 0"/>
-        <inertia ixx="0.001" ixy="0" ixz="0" iyy="0.001" iyz="0" izz="0.001"/>
-      </inertial>
     </link>
     <!-- Lidar -->
@@ -96,6 +55,7 @@
       <origin xyz="0.34 0 0.19" rpy="0 0 0" />
     </joint>
+    </xacro:macro>
     <!-- Wheel -->
-    <xacro:macro name="wheel" params="prefix y_reflect x_reflect ">
+    <xacro:macro name="wheel" params="prefix y_reflect x_reflect x_axis_rotation">
         <link name="${prefix}_wheel">
             <visual>
@@ -115,13 +75,14 @@
             </collision>
         </link>
-        <joint name="base_to_${prefix}_wheel" type="conti">
+        <joint name="base_to_${prefix}_wheel" type="continuous">
             <parent link="base_link"/>
             <child link="${prefix}_wheel"/>
-            <origin xyz="${y_reflect * } ${x_reflect * } 0" rpy/>
+            <axis xyz="0 0 1"/>
+            <origin xyz="${y_reflect * 0.230631} ${x_reflect * 0.22735} 0" rpy=" ${x_axis_rotation * 1.57079632679} 0 0"/>
         </joint>
-    </xacro:macro>
-    <xacro:wheel prefix="front_right" y_reflect="0.5" x_reflect="0.5"/>
-    <xacro:wheel prefix="front_left" y_reflect="0.5" x_reflect="0.5"/>
-    <xacro:wheel prefix="rear_right" y_reflect="0.5" x_reflect="0.5"/>
-    <xacro:wheel prefix="rear_left" y_reflect="0.5" x_reflect="0.5"/>
-</robot>
+     </xacro:macro>
+     <xacro:wheel prefix="front_left" y_reflect="1" x_reflect="1" x_axis_rotation="-1"/>
+     <xacro:wheel prefix="front_right" y_reflect="1" x_reflect="-1" x_axis_rotation="1"/>
+     <xacro:wheel prefix="rear_left" y_reflect="-1" x_reflect="1" x_axis_rotation="-1"/>
+     <xacro:wheel prefix="rear_right" y_reflect="-1" x_reflect="-1" x_axis_rotation="1"/>
+  </robot>

Commit message: Sara's new base/right dimensions/4 wheels added succesfully

File: sara_description/urdf/base_v1/base.urdf.xacro (robot description, xacro)
@@ -9,5 +9,8 @@
             <mesh filename="package://sara_description/meshes/base.STL" scale="0.001 0.001 0.001"/>
          </geometry>
-         <origin xyz="0 0 0" rpy="-1.57 0 1.57"/>
+         <origin xyz="0.295 -0.250 0.85635" rpy="-1.57 0 1.57"/>
+         <material name="blue">
+            <color rgba="0 0 1 1"/>
+         </material>
       </visual>
       <collision>
@@ -15,15 +18,6 @@
             <mesh filename="package://sara_description/meshes/base.STL" scale="0.001 0.001 0.001"/>
          </geometry>
-         <origin xyz="0 0 0" rpy="0 0 0"/>
+         <origin xyz="0.295 -0.250 0.85635" rpy="-1.57 0 1.57"/>
       </collision>
-    </link>
-    <joint name="${name}_spine_joint" type="fixed">
-      <parent link="base_link"/>
-      <child link="spine_link"/>
-      <origin xyz="0 0 0" rpy="0 0 0" />
-      <axis xyz="0 0 0" />
-    </joint>
-  <!-- Lien entre le torse et la colonne vertebrale -->
-    <link name="spine_link">
     </link>
     <!-- Lidar -->
@@ -56,33 +50,3 @@
     </joint>
     </xacro:macro>
-    <!-- Wheel -->
-    <xacro:macro name="wheel" params="prefix y_reflect x_reflect x_axis_rotation">
-        <link name="${prefix}_wheel">
-            <visual>
-                <geometry>
-                    <cylinder length="0.04" radius="0.15"/>
-                </geometry>
-                <origin xyz="0 0 0" rpy="0 0 0"/>
-                <material name="black">
-                    <color rgba="0 0 0 0"/>
-                </material>
-            </visual>
-            <collision>
-                <geometry>
-                    <cylinder length="0.04" radius="0.15"/>
-                </geometry>
-                <origin xyz="0 0 0" rpy="0 0 0"/>
-            </collision>
-        </link>
-        <joint name="base_to_${prefix}_wheel" type="continuous">
-            <parent link="base_link"/>
-            <child link="${prefix}_wheel"/>
-            <axis xyz="0 0 1"/>
-            <origin xyz="${y_reflect * 0.230631} ${x_reflect * 0.22735} 0" rpy=" ${x_axis_rotation * 1.57079632679} 0 0"/>
-        </joint>
-     </xacro:macro>
-     <xacro:wheel prefix="front_left" y_reflect="1" x_reflect="1" x_axis_rotation="-1"/>
-     <xacro:wheel prefix="front_right" y_reflect="1" x_reflect="-1" x_axis_rotation="1"/>
-     <xacro:wheel prefix="rear_left" y_reflect="-1" x_reflect="1" x_axis_rotation="-1"/>
-     <xacro:wheel prefix="rear_right" y_reflect="-1" x_reflect="-1" x_axis_rotation="1"/>
   </robot>

File: sara_description/urdf/sara.urdf.xacro (robot description, xacro)
@@ -8,8 +8,11 @@
     <xacro:include filename="$(find sara_description)/urdf/arm_v1/arm.urdf.xacro"/>
     <xacro:include filename="$(find sara_description)/urdf/base_v1/base.urdf.xacro"/>
+    <xacro:include filename="$(find sara_description)/urdf/wheels_v1/wheels.urdf.xacro"/>
+    <!-- Wheels -->
+    <xacro:sara_wheels_v1 name="wheels" parent="base"/>
     <!-- Base -->
     <xacro:sara_base_v1 name="base" parent=""/>
     <!-- Torso -->
-    <xacro:sara_torso_v1 name="torso" parent="spine"/>
+    <xacro:sara_torso_v1 name="torso" parent="base"/>
     <!-- Neck -->
     <xacro:sara_neck_v1 name="neck" parent="torso"/>

File: sara_description/urdf/torso_v1/torso.urdf.xacro (robot description, xacro)
@@ -30,5 +30,5 @@
          <child link="${name}_link"/>
          <limit effort="1000.0" lower="0" upper="0.5" velocity="0.2"/>
-         <origin xyz="0 0 1.112" rpy="0 0 0" />
+         <origin xyz="0.199974 0 0.85635" rpy="0 0 0" />
          <axis xyz="0 0 1" />
     </joint>

Commit message: updated lidar link

File: sara_description/urdf/base_v1/base.urdf.xacro (robot description, xacro)
@@ -11,5 +11,5 @@
          <origin xyz="0.295 -0.250 0.85635" rpy="-1.57 0 1.57"/>
          <material name="blue">
-            <color rgba="0 0 1 1"/>
+            <color rgba="1 0 1 1"/>
          </material>
       </visual>
@@ -25,7 +25,7 @@
       <visual>
         <geometry>
-          <cylinder length="0.1" radius="0.03"/>
+          <cylinder length="0.085" radius="0.03"/>
         </geometry>
-        <origin xyz="0 0 0" rpy="0 0 0"/>
+        <origin xyz="0 0 0.0425" rpy="0 0 0"/>
         <material name="orange">
           <color rgba="1 0.5 0 1"/>
@@ -34,5 +34,5 @@
       <collision>
         <geometry>
-          <cylinder length="0.1" radius="0.03"/>
+          <cylinder length="0.085" radius="0.03"/>
         </geometry>
         <origin xyz="0 0 0" rpy="0 0 0"/>
@@ -47,5 +47,5 @@
       <parent link="base_link"/>
       <child link="lidar_link"/>
-      <origin xyz="0.34 0 0.19" rpy="0 0 0" />
+      <origin xyz="0.2516879 0 -0.0288348" rpy="0 0 0" />
     </joint>
     </xacro:macro>

Commit message: Fixed wheels xacro macro/Unified color for base

File: sara_description/urdf/base_v1/base.urdf.xacro (robot description, xacro)
@@ -10,6 +10,6 @@
          </geometry>
          <origin xyz="0.295 -0.250 0.85635" rpy="-1.57 0 1.57"/>
-         <material name="blue">
-            <color rgba="1 0 1 1"/>
+         <material name="black">
+               <color rgba="0.12 0.12 0.12 1"/>
          </material>
       </visual>

File: sara_description/urdf/sara.urdf.xacro (robot description, xacro)
@@ -5,12 +5,12 @@
     <xacro:include filename="$(find sara_description)/urdf/neck_v1/neck.urdf.xacro"/>
     <xacro:include filename="$(find sara_description)/urdf/head_v1/head.urdf.xacro"/>
-    <xacro:include filename="$(find sara_description)/urdf/robotiq_c2_model/robotiq_c2_model_macro.xacro"/>
+    <xacro:include filename="$(find sara_description)/urdf/grasp_v1/robotiq_c2_model_macro.xacro"/>
     <xacro:include filename="$(find sara_description)/urdf/arm_v1/arm.urdf.xacro"/>
     <xacro:include filename="$(find sara_description)/urdf/base_v1/base.urdf.xacro"/>
     <xacro:include filename="$(find sara_description)/urdf/wheels_v1/wheels.urdf.xacro"/>
+    <!-- Base -->
+    <xacro:sara_base_v1 name="base" parent=""/>
     <!-- Wheels -->
     <xacro:sara_wheels_v1 name="wheels" parent="base"/>
-    <!-- Base -->
-    <xacro:sara_base_v1 name="base" parent=""/>
     <!-- Torso -->
     <xacro:sara_torso_v1 name="torso" parent="base"/>
@@ -22,4 +22,4 @@
     <xacro:sara_arm_v1 name="arm" parent="torso" end_effector="robotiq_85_base"/>
     <!-- End Effector -->
-    <xacro:robotiq_c2_model prefix=""/>
+    <xacro:sara_grasp_v1 prefix=""/>
 </robot>

Commit message: Urdf fully functionnal

File: sara_description/urdf/base_v1/base.urdf.xacro (robot description, xacro)
@@ -14,4 +14,13 @@
          </material>
       </visual>
+      <visual>
+         <geometry>
+              <box size="0.4 0.35635 0.454"/>
+         </geometry>
+         <origin xyz="-0.055 0 0.227" rpy="0 0 0"/>
+         <material name="black">
+               <color rgba="0.12 0.12 0.12 1"/>
+         </material>
+      </visual>
       <collision>
          <geometry>
@@ -19,4 +28,10 @@
          </geometry>
          <origin xyz="0.295 -0.250 0.85635" rpy="-1.57 0 1.57"/>
+      </collision>
+      <collision>
+        <geometry>
+             <box size="0.4 0.35635 0.454"/>
+        </geometry>
+        <origin xyz="-0.055 0 0.227" rpy="0 0 0"/>
       </collision>
     </link>
